File: EAGLE/Power.Board/Power.Board.brd (EAGLE design)
At the start: 160 x 100 mm, 11 parts, among them X1 MSTBA4, X2 MSTBA10

Commit message: 20180424
Parts:
- moved JP7 35.4 mm to (111.7, 31.7)
- moved JP1 31.2 mm to (106.7, 45.7)
- moved JP9 24.1 mm to (111.7, 14.0)
- moved JP4 18.3 mm to (63.0, 31.7)
- moved JP6 15.0 mm to (71.7, 31.7)
- moved X2 14.5 mm to (40.6, 47.0)
- moved X1 1.26 mm to (5.08, 22.9)
- moved JP5 0.24 mm to (63.0, 14.0)
- moved JP2 0.07 mm to (23.0, 31.7)
Routing:
- net GND: track 0.00 -> 255.8 mm
- net +36V: track 0.00 -> 156.9 mm
- net N$4: track 0.00 -> 51.3 mm
- net +48V: track 0.00 -> 24.1 mm
- net N$5: track 0.00 -> 15.2 mm
Changed lines of the file:
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@@
 <setting verticaltext="up"/>
 </settings>
-<grid distance="0.1" unitdist="mm" unit="mm" style="lines" multiple="1" display="yes" altdistance="0.025" altunitdist="inch" altunit="inch"/>
+<grid distance="0.05" unitdist="inch" unit="mm" style="dots" multiple="1" display="yes" altdistance="0.025" altunitdist="inch" altunit="mm"/>
 <layers>
 <layer number="1" name="Top" color="4" fill="1" visible="yes" active="yes"/>
@@
 <wire x1="160" y1="100" x2="0" y2="100" width="0" layer="20"/>
 <wire x1="0" y1="100" x2="0" y2="0" width="0" layer="20"/>
+<dimension x1="23" y1="31.7" x2="23" y2="14" x3="30.3" y3="22.85" textsize="1.778" layer="16"/>
+<dimension x1="23" y1="14" x2="63" y2="14" x3="43" y3="10.2" textsize="1.778" layer="16"/>
+<wire x1="21" y1="12" x2="65" y2="12" width="0.4064" layer="21"/>
+<wire x1="65" y1="12" x2="65" y2="33.7" width="0.4064" layer="21"/>
+<wire x1="65" y1="33.7" x2="21" y2="33.7" width="0.4064" layer="21"/>
+<wire x1="21" y1="33.7" x2="21" y2="12" width="0.4064" layer="21"/>
+<wire x1="69.7" y1="33.7" x2="69.7" y2="12" width="0.4064" layer="21"/>
+<wire x1="113.7" y1="33.7" x2="69.7" y2="33.7" width="0.4064" layer="21"/>
+<wire x1="69.7" y1="12" x2="113.7" y2="12" width="0.4064" layer="21"/>
+<wire x1="113.7" y1="12" x2="113.7" y2="33.7" width="0.4064" layer="21"/>
 </plain>
 <attributes>
@@
 </autorouter>
 <elements>
-<element name="X1" library="con-phoenix-508" package="MSTBA4" value="MSTBA4" x="5.08" y="21.59" rot="R270"/>
-<element name="X2" library="con-phoenix-508" package="MSTBA10" value="MSTBA10" x="44.45" y="60.96" rot="R180"/>
-<element name="JP1" library="pinhead" package="1X03/90" value="" x="78.74" y="59.69"/>
-<element name="JP2" library="pinhead" package="1X01" value="" x="23.04" y="31.64"/>
-<element name="JP3" library="pinhead" package="1X01" value="" x="22.96" y="13.97"/>
-<element name="JP4" library="pinhead" package="1X01" value="" x="46.99" y="40.64"/>
-<element name="JP5" library="pinhead" package="1X01" value="" x="63.06" y="13.77"/>
-<element name="JP6" library="pinhead" package="1X01" value="" x="59.69" y="40.64"/>
-<element name="JP7" library="pinhead" package="1X01" value="" x="77.47" y="40.64"/>
-<element name="JP8" library="pinhead" package="1X01" value="" x="71.7" y="13.97"/>
-<element name="JP9" library="pinhead" package="1X01" value="" x="87.63" y="13.97"/>
+<element name="X1" library="con-phoenix-508" package="MSTBA4" value="MSTBA4" x="5.08" y="22.85" rot="R270"/>
+<element name="X2" library="con-phoenix-508" package="MSTBA10" value="MSTBA10" x="40.64" y="46.99" rot="R180"/>
+<element name="JP1" library="pinhead" package="1X03/90" value="" x="106.68" y="45.72"/>
+<element name="JP2" library="pinhead" package="1X01" value="" x="23" y="31.7"/>
+<element name="JP3" library="pinhead" package="1X01" value="" x="23" y="14"/>
+<element name="JP4" library="pinhead" package="1X01" value="" x="63" y="31.7"/>
+<element name="JP5" library="pinhead" package="1X01" value="" x="63" y="14"/>
+<element name="JP6" library="pinhead" package="1X01" value="" x="71.7" y="31.7"/>
+<element name="JP7" library="pinhead" package="1X01" value="" x="111.7" y="31.7"/>
+<element name="JP8" library="pinhead" package="1X01" value="" x="71.7" y="14"/>
+<element name="JP9" library="pinhead" package="1X01" value="" x="111.7" y="14"/>
 </elements>
 <signals>
@@
 <contactref element="X2" pad="2"/>
 <contactref element="X1" pad="2"/>
-<wire x1="31.75" y1="55.88" x2="21.59" y2="55.88" width="0" layer="19" extent="1-1"/>
-<wire x1="41.91" y1="55.88" x2="31.75" y2="55.88" width="0" layer="19" extent="1-1"/>
-<wire x1="52.07" y1="55.88" x2="41.91" y2="55.88" width="0" layer="19" extent="1-1"/>
-<wire x1="62.23" y1="55.88" x2="52.07" y2="55.88" width="0" layer="19" extent="1-1"/>
-<wire x1="10.16" y1="13.97" x2="62.23" y2="55.88" width="0" layer="19" extent="1-1"/>
-<wire x1="10.16" y1="24.13" x2="10.16" y2="13.97" width="0" layer="19" extent="1-1"/>
-<wire x1="22.96" y1="13.97" x2="10.16" y2="13.97" width="0" layer="19" extent="1-1"/>
-<wire x1="63.06" y1="13.77" x2="22.96" y2="13.97" width="0" layer="19" extent="1-1"/>
-<wire x1="71.7" y1="13.97" x2="63.06" y2="13.77" width="0" layer="19" extent="1-1"/>
-<wire x1="87.63" y1="13.97" x2="71.7" y2="13.97" width="0" layer="19" extent="1-1"/>
-<wire x1="81.28" y1="55.88" x2="71.7" y2="13.97" width="0" layer="19" extent="1-1"/>
+<wire x1="17.78" y1="41.91" x2="17.78" y2="46.99" width="3.81" layer="16"/>
+<wire x1="17.78" y1="46.99" x2="27.94" y2="46.99" width="3.81" layer="16"/>
+<wire x1="27.94" y1="41.91" x2="27.94" y2="46.99" width="3.81" layer="16"/>
+<wire x1="27.94" y1="46.99" x2="38.1" y2="46.99" width="3.81" layer="16"/>
+<wire x1="58.42" y1="41.91" x2="58.42" y2="46.99" width="3.81" layer="16"/>
+<wire x1="58.42" y1="46.99" x2="48.26" y2="46.99" width="3.81" layer="16"/>
+<wire x1="48.26" y1="41.91" x2="48.26" y2="46.99" width="3.81" layer="16"/>
+<wire x1="48.26" y1="46.99" x2="38.1" y2="46.99" width="3.81" layer="16"/>
+<wire x1="38.1" y1="46.99" x2="38.1" y2="41.91" width="3.81" layer="16"/>
+<wire x1="10.16" y1="15.23" x2="5.08" y2="15.23" width="3.81" layer="16"/>
+<wire x1="5.08" y1="15.23" x2="5.08" y2="25.4" width="3.81" layer="16"/>
+<wire x1="5.08" y1="25.4" x2="10.16" y2="25.4" width="3.81" layer="16"/>
+<wire x1="10.16" y1="25.4" x2="10.16" y2="25.39" width="2.54" layer="16"/>
+<wire x1="17.78" y1="41.91" x2="5.08" y2="41.91" width="3.81" layer="16"/>
+<wire x1="5.08" y1="41.91" x2="5.08" y2="25.4" width="3.81" layer="16"/>
+<wire x1="23" y1="14" x2="63" y2="14" width="2.54" layer="16"/>
+<wire x1="63" y1="14" x2="71.7" y2="14" width="2.54" layer="16"/>
+<wire x1="71.7" y1="14" x2="111.7" y2="14" width="2.54" layer="16"/>
+<wire x1="23" y1="14" x2="17.75" y2="14" width="2.54" layer="16"/>
+<wire x1="17.75" y1="14" x2="16.51" y2="15.24" width="2.54" layer="16"/>
+<wire x1="16.51" y1="15.24" x2="10.17" y2="15.24" width="2.54" layer="16"/>
+<wire x1="10.17" y1="15.24" x2="10.16" y2="15.23" width="1.27" layer="16"/>
+<wire x1="109.22" y1="41.91" x2="115.57" y2="41.91" width="1.27" layer="16"/>
+<wire x1="115.57" y1="41.91" x2="115.57" y2="13.97" width="1.27" layer="16"/>
+<wire x1="115.57" y1="13.97" x2="111.7" y2="13.97" width="1.27" layer="16"/>
+<wire x1="111.7" y1="13.97" x2="111.7" y2="14" width="1.27" layer="16"/>
 </signal>
 <signal name="+36V">
@@
 <contactref element="X2" pad="1"/>
 <contactref element="X1" pad="3"/>
-<wire x1="46.99" y1="55.88" x2="36.83" y2="55.88" width="0" layer="19" extent="1-1"/>
-<wire x1="57.15" y1="55.88" x2="46.99" y2="55.88" width="0" layer="19" extent="1-1"/>
-<wire x1="67.31" y1="55.88" x2="57.15" y2="55.88" width="0" layer="19" extent="1-1"/>
-<wire x1="10.16" y1="19.05" x2="67.31" y2="55.88" width="0" layer="19" extent="1-1"/>
-<wire x1="59.69" y1="40.64" x2="10.16" y2="19.05" width="0" layer="19" extent="1-1"/>
-<wire x1="23.04" y1="31.64" x2="59.69" y2="40.64" width="0" layer="19" extent="1-1"/>
+<wire x1="33.02" y1="41.91" x2="33.02" y2="36.83" width="2.54" layer="16"/>
+<wire x1="33.02" y1="36.83" x2="43.18" y2="36.83" width="3.81" layer="16"/>
+<wire x1="43.18" y1="41.91" x2="43.18" y2="36.83" width="3.81" layer="16"/>
+<wire x1="43.18" y1="36.83" x2="53.34" y2="36.83" width="3.81" layer="16"/>
+<wire x1="53.34" y1="41.91" x2="53.34" y2="36.83" width="3.81" layer="16"/>
+<wire x1="53.34" y1="36.83" x2="63.5" y2="36.83" width="3.81" layer="16"/>
+<wire x1="63.5" y1="36.83" x2="63.5" y2="41.91" width="3.81" layer="16"/>
+<wire x1="10.16" y1="20.31" x2="22.86" y2="20.31" width="3.81" layer="16"/>
+<wire x1="22.86" y1="20.31" x2="33.02" y2="20.31" width="3.81" layer="16"/>
+<wire x1="33.02" y1="20.31" x2="33.02" y2="31.75" width="3.81" layer="16"/>
+<wire x1="33.02" y1="31.75" x2="33.02" y2="41.91" width="3.81" layer="16"/>
+<wire x1="33.02" y1="31.7" x2="33.02" y2="31.75" width="1.27" layer="16"/>
+<wire x1="71.7" y1="31.7" x2="71.7" y2="20.31" width="2.54" layer="16"/>
+<wire x1="71.7" y1="20.31" x2="33.02" y2="20.31" width="2.54" layer="16"/>
+<wire x1="23" y1="31.7" x2="22.86" y2="31.7" width="1.27" layer="16"/>
+<wire x1="22.86" y1="31.7" x2="22.86" y2="20.31" width="2.54" layer="16"/>
 </signal>
 <signal name="N$4">
 <contactref element="JP4" pad="1"/>
 <contactref element="JP1" pad="1"/>
-<wire x1="46.99" y1="40.64" x2="76.2" y2="55.88" width="0" layer="19" extent="1-1"/>
+<wire x1="63" y1="31.7" x2="67.31" y2="31.7" width="1.27" layer="16"/>
+<wire x1="67.31" y1="31.7" x2="67.31" y2="35.56" width="1.27" layer="16"/>
+<wire x1="67.31" y1="35.56" x2="104.14" y2="35.56" width="1.27" layer="16"/>
+<wire x1="104.14" y1="35.56" x2="104.14" y2="41.91" width="1.27" layer="16"/>
 </signal>
 <signal name="N$5">
 <contactref element="JP7" pad="1"/>
 <contactref element="JP1" pad="2"/>
-<wire x1="77.47" y1="40.64" x2="78.74" y2="55.88" width="0" layer="19" extent="1-1"/>
+<wire x1="111.7" y1="31.7" x2="106.68" y2="31.7" width="1.27" layer="16"/>
+<wire x1="106.68" y1="31.7" x2="106.68" y2="41.91" width="1.27" layer="16"/>
 </signal>
 <signal name="+48V">
 <contactref element="X2" pad="9"/>
 <contactref element="X1" pad="1"/>
-<wire x1="10.16" y1="29.21" x2="26.67" y2="55.88" width="0" layer="19" extent="1-1"/>
+<wire x1="10.16" y1="30.47" x2="10.16" y2="36.83" width="3.81" layer="16"/>
+<wire x1="10.16" y1="36.83" x2="22.86" y2="36.83" width="3.81" layer="16"/>
+<wire x1="22.86" y1="36.83" x2="22.86" y2="41.91" width="3.81" layer="16"/>
 </signal>
 </signals>

Commit message: PCB-GCODE-3.6.0.4 added
Parts:
- moved JP1 3.00 mm to (106.7, 42.7)
- moved JP2 3.00 mm to (23.0, 28.7)
- moved JP3 3.00 mm to (23.0, 11.0)
- moved JP4 3.00 mm to (63.0, 28.7)
- moved JP5 3.00 mm to (63.0, 11.0)
- moved JP6 3.00 mm to (71.7, 28.7)
- moved JP7 3.00 mm to (111.7, 28.7)
- moved JP8 3.00 mm to (71.7, 11.0)
- moved JP9 3.00 mm to (111.7, 11.0)
- moved X1 3.00 mm to (5.08, 19.9)
- moved X2 3.00 mm to (40.6, 44.0)
Other:
- board size 160 x 100 mm -> 120 x 49 mm
