File: EAGLE/Control.Board/Control.Board.brd (EAGLE design)
At the start: 160 x 100 mm, 35 parts, among them J1 AVR_SPI_PROG_3X2PTH, U1.X LTV817LTV817S, U1.Y LTV817LTV817S, U1.Z LTV817LTV817S, U2.X LTV817LTV817S, U2.Y LTV817LTV817S, U2.Z LTV817LTV817S

Commit message: 20180416
Parts:
- added PWR-STEPPERS: MSTBA8, con-phoenix-508:MSTBA8
- added STEPPER-CTRL-X1, STEPPER-CTRL-X3, STEPPER-CTRL-Y, STEPPER-CTRL-Z, X6: MSTBA6, con-phoenix-508:MSTBA6
Connections:
- new net +36V: PWR-STEPPERS.1, PWR-STEPPERS.3, PWR-STEPPERS.5, PWR-STEPPERS.7, X6.3
- new net +48V: X6.5
- net +12V: now also X6.1
- net GND: now also PWR-STEPPERS.2, PWR-STEPPERS.4, PWR-STEPPERS.6, PWR-STEPPERS.8, X6.2, X6.4, X6.6
Changed lines of the file:
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@@
 <element name="LED2.Z" library="led" package="CHIPLED_0805" value="" x="-27.94" y="-143.51"/>
 <element name="R1" library="rcl" package="M1206" value="" x="-27.94" y="-154.94"/>
+<element name="STEPPER-CTRL-X3" library="con-phoenix-508" package="MSTBA6" value="MSTBA6" x="-13.97" y="-167.64"/>
+<element name="STEPPER-CTRL-X1" library="con-phoenix-508" package="MSTBA6" value="MSTBA6" x="-13.97" y="-182.88"/>
+<element name="STEPPER-CTRL-Y" library="con-phoenix-508" package="MSTBA6" value="MSTBA6" x="-13.97" y="-198.12"/>
+<element name="STEPPER-CTRL-Z" library="con-phoenix-508" package="MSTBA6" value="MSTBA6" x="-13.97" y="-213.36"/>
+<element name="PWR-STEPPERS" library="con-phoenix-508" package="MSTBA8" value="MSTBA8" x="-8.89" y="-228.6"/>
+<element name="X6" library="con-phoenix-508" package="MSTBA6" value="MSTBA6" x="-13.97" y="-243.84"/>
 </elements>
 <signals>
@@
 <contactref element="U1.Z" pad="3"/>
 <contactref element="U2.Z" pad="3"/>
+<contactref element="X6" pad="2"/>
+<contactref element="X6" pad="4"/>
+<contactref element="X6" pad="6"/>
+<contactref element="PWR-STEPPERS" pad="8"/>
+<contactref element="PWR-STEPPERS" pad="6"/>
+<contactref element="PWR-STEPPERS" pad="4"/>
+<contactref element="PWR-STEPPERS" pad="2"/>
+<wire x1="-1.27" y1="-238.76" x2="-11.43" y2="-238.76" width="0" layer="19" extent="1-1"/>
+<wire x1="-21.59" y1="-238.76" x2="-11.43" y2="-238.76" width="0" layer="19" extent="1-1"/>
+<wire x1="-21.59" y1="-223.52" x2="-21.59" y2="-238.76" width="0" layer="19" extent="1-1"/>
+<wire x1="-11.43" y1="-223.52" x2="-21.59" y2="-223.52" width="0" layer="19" extent="1-1"/>
+<wire x1="-1.27" y1="-223.52" x2="-11.43" y2="-223.52" width="0" layer="19" extent="1-1"/>
+<wire x1="8.89" y1="-223.52" x2="-1.27" y2="-223.52" width="0" layer="19" extent="1-1"/>
+<wire x1="-22.86" y1="-149.86" x2="-21.59" y2="-223.52" width="0" layer="19" extent="1-1"/>
 <wire x1="-15.24" y1="-149.86" x2="-22.86" y2="-149.86" width="0" layer="19" extent="1-1"/>
 <wire x1="-16.51" y1="-135.58" x2="-15.24" y2="-149.86" width="0" layer="19" extent="1-1"/>
@@
 <contactref element="JP.LIMIT.Z" pad="1"/>
 <contactref element="JP.LIMIT.Z" pad="4"/>
+<contactref element="X6" pad="1"/>
 <wire x1="-20.32" y1="-149.86" x2="-27.94" y2="-149.86" width="0" layer="19" extent="1-1"/>
 <wire x1="-27.94" y1="-116.84" x2="-27.94" y2="-149.86" width="0" layer="19" extent="1-1"/>
 <wire x1="-20.32" y1="-116.84" x2="-27.94" y2="-116.84" width="0" layer="19" extent="1-1"/>
+<wire x1="-26.67" y1="-238.76" x2="-27.94" y2="-149.86" width="0" layer="19" extent="1-1"/>
 <wire x1="81.28" y1="40.64" x2="-20.32" y2="-116.84" width="0" layer="19" extent="1-1"/>
 <wire x1="88.9" y1="40.64" x2="81.28" y2="40.64" width="0" layer="19" extent="1-1"/>
@@
 <wire x1="-10.16" y1="-124.68" x2="-27.94" y2="-135.58" width="0" layer="19" extent="1-1"/>
 </signal>
+<signal name="+36V">
+<contactref element="X6" pad="3"/>
+<contactref element="PWR-STEPPERS" pad="5"/>
+<contactref element="PWR-STEPPERS" pad="3"/>
+<contactref element="PWR-STEPPERS" pad="7"/>
+<contactref element="PWR-STEPPERS" pad="1"/>
+<wire x1="-16.51" y1="-223.52" x2="-26.67" y2="-223.52" width="0" layer="19" extent="1-1"/>
+<wire x1="-6.35" y1="-223.52" x2="-16.51" y2="-223.52" width="0" layer="19" extent="1-1"/>
+<wire x1="3.81" y1="-223.52" x2="-6.35" y2="-223.52" width="0" layer="19" extent="1-1"/>
+<wire x1="-16.51" y1="-238.76" x2="-16.51" y2="-223.52" width="0" layer="19" extent="1-1"/>
+</signal>
+<signal name="+48V">
+<contactref element="X6" pad="5"/>
+</signal>
 </signals>

Commit message: 20180427
Parts:
- removed C2: (no value), rcl:C050-035X075
- removed PWR-STEPPERS: MSTBA8, con-phoenix-508:MSTBA8
- removed Q2: (no value), crystal:HC49/S
- removed X6: MSTBA6, con-phoenix-508:MSTBA6
- renumbered STEPPER-CTRL-X3 to STEPPER-CTRL-X2
Connections:
- removed net +36V: PWR-STEPPERS.1, PWR-STEPPERS.3, PWR-STEPPERS.5, PWR-STEPPERS.7, X6.3
- removed net +48V: X6.5
- net +12V: no longer X6.1
- net GND: no longer PWR-STEPPERS.2, PWR-STEPPERS.4, PWR-STEPPERS.6, PWR-STEPPERS.8, X6.2, X6.4, X6.6
- net MEGA2560.D0.RXD0: no longer C2.1
Changed lines of the file:
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@@
 <elements>
 <element name="JP.LIMIT.X" library="pinhead" package="1X06" value="" x="87.63" y="40.64"/>
-<element name="Q2" library="crystal" package="HC49/S" value="" x="72.39" y="34.29">
-<attribute name="OC_NEWARK" value="unknown" x="138.43" y="3.81" size="1.778" layer="27" display="off"/>
-<attribute name="MPN" value="" x="138.43" y="3.81" size="1.778" layer="27" display="off"/>
-<attribute name="MF" value="" x="138.43" y="3.81" size="1.778" layer="27" display="off"/>
-<attribute name="OC_FARNELL" value="1667008" x="138.43" y="3.81" size="1.778" layer="27" display="off"/>
-</element>
-<element name="C2" library="rcl" package="C050-035X075" value="" x="68.58" y="41.91"/>
 <element name="JP.MEGA2560.POWER" library="pinhead" package="1X08" value="" x="5.08" y="69.85" rot="R270"/>
 <element name="JP.MEGA2560.ANALOG.LOW" library="pinhead" package="1X08" value="" x="5.08" y="46.99" rot="R270"/>
@@
 <element name="LED2.Z" library="led" package="CHIPLED_0805" value="" x="-27.94" y="-143.51"/>
 <element name="R1" library="rcl" package="M1206" value="" x="-27.94" y="-154.94"/>
-<element name="STEPPER-CTRL-X3" library="con-phoenix-508" package="MSTBA6" value="MSTBA6" x="-13.97" y="-167.64"/>
+<element name="STEPPER-CTRL-X2" library="con-phoenix-508" package="MSTBA6" value="MSTBA6" x="-13.97" y="-167.64"/>
 <element name="STEPPER-CTRL-X1" library="con-phoenix-508" package="MSTBA6" value="MSTBA6" x="-13.97" y="-182.88"/>
 <element name="STEPPER-CTRL-Y" library="con-phoenix-508" package="MSTBA6" value="MSTBA6" x="-13.97" y="-198.12"/>
 <element name="STEPPER-CTRL-Z" library="con-phoenix-508" package="MSTBA6" value="MSTBA6" x="-13.97" y="-213.36"/>
-<element name="PWR-STEPPERS" library="con-phoenix-508" package="MSTBA8" value="MSTBA8" x="-8.89" y="-228.6"/>
-<element name="X6" library="con-phoenix-508" package="MSTBA6" value="MSTBA6" x="-13.97" y="-243.84"/>
 </elements>
 <signals>
@@
 <contactref element="U1.Z" pad="3"/>
 <contactref element="U2.Z" pad="3"/>
-<contactref element="X6" pad="2"/>
-<contactref element="X6" pad="4"/>
-<contactref element="X6" pad="6"/>
-<contactref element="PWR-STEPPERS" pad="8"/>
-<contactref element="PWR-STEPPERS" pad="6"/>
-<contactref element="PWR-STEPPERS" pad="4"/>
-<contactref element="PWR-STEPPERS" pad="2"/>
-<wire x1="-1.27" y1="-238.76" x2="-11.43" y2="-238.76" width="0" layer="19" extent="1-1"/>
-<wire x1="-21.59" y1="-238.76" x2="-11.43" y2="-238.76" width="0" layer="19" extent="1-1"/>
-<wire x1="-21.59" y1="-223.52" x2="-21.59" y2="-238.76" width="0" layer="19" extent="1-1"/>
-<wire x1="-11.43" y1="-223.52" x2="-21.59" y2="-223.52" width="0" layer="19" extent="1-1"/>
-<wire x1="-1.27" y1="-223.52" x2="-11.43" y2="-223.52" width="0" layer="19" extent="1-1"/>
-<wire x1="8.89" y1="-223.52" x2="-1.27" y2="-223.52" width="0" layer="19" extent="1-1"/>
-<wire x1="-22.86" y1="-149.86" x2="-21.59" y2="-223.52" width="0" layer="19" extent="1-1"/>
 <wire x1="-15.24" y1="-149.86" x2="-22.86" y2="-149.86" width="0" layer="19" extent="1-1"/>
 <wire x1="-16.51" y1="-135.58" x2="-15.24" y2="-149.86" width="0" layer="19" extent="1-1"/>
@@
 <contactref element="JP.LIMIT.Z" pad="1"/>
 <contactref element="JP.LIMIT.Z" pad="4"/>
-<contactref element="X6" pad="1"/>
 <wire x1="-20.32" y1="-149.86" x2="-27.94" y2="-149.86" width="0" layer="19" extent="1-1"/>
 <wire x1="-27.94" y1="-116.84" x2="-27.94" y2="-149.86" width="0" layer="19" extent="1-1"/>
 <wire x1="-20.32" y1="-116.84" x2="-27.94" y2="-116.84" width="0" layer="19" extent="1-1"/>
-<wire x1="-26.67" y1="-238.76" x2="-27.94" y2="-149.86" width="0" layer="19" extent="1-1"/>
 <wire x1="81.28" y1="40.64" x2="-20.32" y2="-116.84" width="0" layer="19" extent="1-1"/>
 <wire x1="88.9" y1="40.64" x2="81.28" y2="40.64" width="0" layer="19" extent="1-1"/>
@@
 <signal name="MEGA2560.D0.RXD0">
 <contactref element="JP.MEGA2560.PWM.LOW" pad="8"/>
-<contactref element="C2" pad="1"/>
-<wire x1="66.04" y1="41.91" x2="53.34" y2="43.18" width="0" layer="19" extent="1-1"/>
 </signal>
 <signal name="MEGA2560.D1.TXD0">
@@
 <wire x1="-10.16" y1="-124.68" x2="-27.94" y2="-135.58" width="0" layer="19" extent="1-1"/>
 </signal>
-<signal name="+36V">
-<contactref element="X6" pad="3"/>
-<contactref element="PWR-STEPPERS" pad="5"/>
-<contactref element="PWR-STEPPERS" pad="3"/>
-<contactref element="PWR-STEPPERS" pad="7"/>
-<contactref element="PWR-STEPPERS" pad="1"/>
-<wire x1="-16.51" y1="-223.52" x2="-26.67" y2="-223.52" width="0" layer="19" extent="1-1"/>
-<wire x1="-6.35" y1="-223.52" x2="-16.51" y2="-223.52" width="0" layer="19" extent="1-1"/>
-<wire x1="3.81" y1="-223.52" x2="-6.35" y2="-223.52" width="0" layer="19" extent="1-1"/>
-<wire x1="-16.51" y1="-238.76" x2="-16.51" y2="-223.52" width="0" layer="19" extent="1-1"/>
-</signal>
-<signal name="+48V">
-<contactref element="X6" pad="5"/>
-</signal>
 </signals>

Commit message: 20180503
Parts:
- added LED1, LED2, LED3, LED4: (no value), led:CHIPLED_1206
- added R2, R3, R4, R5: (no value), rcl:M1206
- added U$1, U$2, U$3, U$4: LTV817LTV817S, net173:DIL4-SMD
- added X1: (no value), con-molex-micro-fit-3_0:43045-0800
Connections:
- new net N$19: LED2.A, X1.P$8
- new net N$20: LED1.A, X1.P$6
- new net N$21: LED3.A, X1.P$4
- new net N$22: LED2.C, R4.1
- new net N$23: R4.2, U$1.1
- new net N$24: R5.2, U$2.1
- new net N$30: LED1.C, R5.1
- new net N$31: LED4.A, X1.P$2
- new net N$32: LED3.C, R3.1
- new net N$33: LED4.C, R2.1
- new net N$34: R2.2, U$4.1
- new net N$35: R3.2, U$3.1
- net +5V: now also X1.P$1, X1.P$3, X1.P$5, X1.P$7
- net GND: now also U$1.2, U$2.2, U$3.2, U$4.2
Changed lines of the file:
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@@
 <element name="STEPPER-CTRL-Y" library="con-phoenix-508" package="MSTBA6" value="MSTBA6" x="-13.97" y="-198.12"/>
 <element name="STEPPER-CTRL-Z" library="con-phoenix-508" package="MSTBA6" value="MSTBA6" x="-13.97" y="-213.36"/>
+<element name="U$1" library="net173" package="DIL4-SMD" value="LTV817LTV817S" x="-35.56" y="-212.09"/>
+<element name="U$2" library="net173" package="DIL4-SMD" value="LTV817LTV817S" x="-44.45" y="-212.09"/>
+<element name="U$3" library="net173" package="DIL4-SMD" value="LTV817LTV817S" x="-53.34" y="-212.09"/>
+<element name="U$4" library="net173" package="DIL4-SMD" value="LTV817LTV817S" x="-62.23" y="-212.09"/>
+<element name="R2" library="rcl" package="M1206" value="" x="-63.5" y="-222.25"/>
+<element name="R3" library="rcl" package="M1206" value="" x="-63.5" y="-227.33"/>
+<element name="R4" library="rcl" package="M1206" value="" x="-63.5" y="-232.41"/>
+<element name="R5" library="rcl" package="M1206" value="" x="-63.5" y="-237.49"/>
+<element name="LED1" library="led" package="CHIPLED_1206" value="" x="-69.85" y="-236.22"/>
+<element name="LED2" library="led" package="CHIPLED_1206" value="" x="-76.2" y="-236.22"/>
+<element name="LED3" library="led" package="CHIPLED_1206" value="" x="-82.55" y="-236.22"/>
+<element name="LED4" library="led" package="CHIPLED_1206" value="" x="-88.9" y="-236.22"/>
+<element name="X1" library="con-molex-micro-fit-3_0" package="43045-0800" value="" x="-82.55" y="-247.65"/>
 </elements>
 <signals>
@@
 <contactref element="U1.Z" pad="3"/>
 <contactref element="U2.Z" pad="3"/>
+<contactref element="U$1" pad="2"/>
+<contactref element="U$4" pad="2"/>
+<contactref element="U$3" pad="2"/>
+<contactref element="U$2" pad="2"/>
+<wire x1="-43.18" y1="-216.86" x2="-34.29" y2="-216.86" width="0" layer="19" extent="1-1"/>
+<wire x1="-52.07" y1="-216.86" x2="-43.18" y2="-216.86" width="0" layer="19" extent="1-1"/>
+<wire x1="-60.96" y1="-216.86" x2="-52.07" y2="-216.86" width="0" layer="19" extent="1-1"/>
+<wire x1="-22.86" y1="-149.86" x2="-34.29" y2="-216.86" width="0" layer="19" extent="1-1"/>
 <wire x1="-15.24" y1="-149.86" x2="-22.86" y2="-149.86" width="0" layer="19" extent="1-1"/>
 <wire x1="-16.51" y1="-135.58" x2="-15.24" y2="-149.86" width="0" layer="19" extent="1-1"/>
@@
 <contactref element="R3.Y" pad="2"/>
 <contactref element="R3.Z" pad="2"/>
+<contactref element="X1" pad="P$1"/>
+<contactref element="X1" pad="P$3"/>
+<contactref element="X1" pad="P$5"/>
+<contactref element="X1" pad="P$7"/>
 <wire x1="-10.48" y1="-106.68" x2="-10.48" y2="-139.7" width="0" layer="19" extent="1-1"/>
 <wire x1="-14.29" y1="-82.55" x2="-10.48" y2="-106.68" width="0" layer="19" extent="1-1"/>
+<wire x1="-78.05" y1="-240.33" x2="-10.48" y2="-139.7" width="0" layer="19" extent="1-1"/>
+<wire x1="-78.05" y1="-243.33" x2="-78.05" y2="-240.33" width="0" layer="19" extent="1-1"/>
+<wire x1="-84.05" y1="-243.33" x2="-78.05" y2="-243.33" width="0" layer="19" extent="1-1"/>
+<wire x1="-84.05" y1="-240.33" x2="-84.05" y2="-243.33" width="0" layer="19" extent="1-1"/>
 </signal>
 <signal name="N$25">
@@
 <wire x1="-10.16" y1="-124.68" x2="-27.94" y2="-135.58" width="0" layer="19" extent="1-1"/>
 </signal>
+<signal name="N$19">
+<contactref element="X1" pad="P$8"/>
+<contactref element="LED2" pad="A"/>
+<wire x1="-76.2" y1="-237.97" x2="-87.05" y2="-240.33" width="0" layer="19" extent="1-1"/>
+</signal>
+<signal name="N$20">
+<contactref element="X1" pad="P$6"/>
+<contactref element="LED1" pad="A"/>
+<wire x1="-69.85" y1="-237.97" x2="-81.05" y2="-240.33" width="0" layer="19" extent="1-1"/>
+</signal>
+<signal name="N$21">
+<contactref element="X1" pad="P$4"/>
+<contactref element="LED3" pad="A"/>
+<wire x1="-82.55" y1="-237.97" x2="-87.05" y2="-243.33" width="0" layer="19" extent="1-1"/>
+</signal>
+<signal name="N$22">
+<contactref element="LED2" pad="C"/>
+<contactref element="R4" pad="1"/>
+<wire x1="-64.9" y1="-232.41" x2="-76.2" y2="-234.47" width="0" layer="19" extent="1-1"/>
+</signal>
+<signal name="N$23">
+<contactref element="R4" pad="2"/>
+<contactref element="U$1" pad="1"/>
+<wire x1="-62.1" y1="-232.41" x2="-36.83" y2="-216.86" width="0" layer="19" extent="1-1"/>
+</signal>
+<signal name="N$24">
+<contactref element="R5" pad="2"/>
+<contactref element="U$2" pad="1"/>
+<wire x1="-45.72" y1="-216.86" x2="-62.1" y2="-237.49" width="0" layer="19" extent="1-1"/>
+</signal>
+<signal name="N$30">
+<contactref element="LED1" pad="C"/>
+<contactref element="R5" pad="1"/>
+<wire x1="-64.9" y1="-237.49" x2="-69.85" y2="-234.47" width="0" layer="19" extent="1-1"/>
+</signal>
+<signal name="N$31">
+<contactref element="LED4" pad="A"/>
+<contactref element="X1" pad="P$2"/>
+<wire x1="-81.05" y1="-243.33" x2="-88.9" y2="-237.97" width="0" layer="19" extent="1-1"/>
+</signal>
+<signal name="N$32">
+<contactref element="LED3" pad="C"/>
+<contactref element="R3" pad="1"/>
+<wire x1="-64.9" y1="-227.33" x2="-82.55" y2="-234.47" width="0" layer="19" extent="1-1"/>
+</signal>
+<signal name="N$33">
+<contactref element="LED4" pad="C"/>
+<contactref element="R2" pad="1"/>
+<wire x1="-64.9" y1="-222.25" x2="-88.9" y2="-234.47" width="0" layer="19" extent="1-1"/>
+</signal>
+<signal name="N$34">
+<contactref element="R2" pad="2"/>
+<contactref element="U$4" pad="1"/>
+<wire x1="-63.5" y1="-216.86" x2="-62.1" y2="-222.25" width="0" layer="19" extent="1-1"/>
+</signal>
+<signal name="N$35">
+<contactref element="R3" pad="2"/>
+<contactref element="U$3" pad="1"/>
+<wire x1="-54.61" y1="-216.86" x2="-62.1" y2="-227.33" width="0" layer="19" extent="1-1"/>
+</signal>
 </signals>

Commit message: 20180503
Parts:
- removed STEPPER-CTRL-X1, STEPPER-CTRL-X2, STEPPER-CTRL-Y, STEPPER-CTRL-Z: MSTBA6, con-phoenix-508:MSTBA6
- added STEPPER-X1, STEPPER-X2, STEPPER-Y, STEPPER-Z: (no value), con-molex-micro-fit-3_0:43045-0600
- R2, R3, R4, R5: value (none) -> 100
Connections:
- net +5V: now also STEPPER-X1.P$1, STEPPER-X1.P$2, STEPPER-X1.P$3, STEPPER-X2.P$1, STEPPER-X2.P$2, STEPPER-X2.P$3, STEPPER-Y.P$1, STEPPER-Y.P$2, STEPPER-Y.P$3, STEPPER-Z.P$1, STEPPER-Z.P$2, STEPPER-Z.P$3, X1.P$2, X1.P$4; no longer X1.P$5, X1.P$7
- net GND: now also U$1.3, U$2.3, U$3.3, U$4.3
- net MEGA2560.A10.CYCLE.START: now also U$3.4
- net MEGA2560.A11.SAFETY.DOOR: now also U$4.4
- net MEGA2560.A8.RESET.ABORT: now also U$1.4
- net MEGA2560.A9.FEED.HOLD: now also U$2.4
- net MEGA2560.D13.STEPPER.EN: now also STEPPER-X1.P$6, STEPPER-X2.P$6, STEPPER-Y.P$6, STEPPER-Z.P$6
- net MEGA2560.D24.STEP.X: now also STEPPER-X1.P$4, STEPPER-X2.P$4
- net MEGA2560.D25.STEP.Y: now also STEPPER-Y.P$4
- net MEGA2560.D26.STEP.Z: now also STEPPER-Z.P$4
- net MEGA2560.D30.DIR.X: now also STEPPER-X1.P$5, STEPPER-X2.P$5
- net MEGA2560.D31.DIR.Y: now also STEPPER-Y.P$5
- net MEGA2560.D32.DIR.Z: now also STEPPER-Z.P$5
- net N$20: now also X1.P$7; no longer X1.P$6
- net N$21: now also X1.P$6; no longer X1.P$4
- net N$31: now also X1.P$5; no longer X1.P$2
