File: EAGLE/Control.Board/Control.Board.sch (EAGLE design)
At the start: 35 parts, among them J1 AVR_SPI_PROG_3X2PTH, U1.X LTV817LTV817S, U1.Y LTV817LTV817S, U1.Z LTV817LTV817S, U2.X LTV817LTV817S, U2.Y LTV817LTV817S, U2.Z LTV817LTV817S

Commit message: 20180416
Parts:
- added PWR-STEPPERS: MSTBA8, con-phoenix-508:MSTBA8
- added STEPPER-CTRL-X1, STEPPER-CTRL-X3, STEPPER-CTRL-Y, STEPPER-CTRL-Z, X6: MSTBA6, con-phoenix-508:MSTBA6
Connections:
- new net +36V: PWR-STEPPERS-1.1, PWR-STEPPERS-3.1, PWR-STEPPERS-5.1, PWR-STEPPERS-7.1, X6-3.1
- new net +48V: X6-5.1
- net +12V: now also X6-1.1
- net GND: now also PWR-STEPPERS-2.1, PWR-STEPPERS-4.1, PWR-STEPPERS-6.1, PWR-STEPPERS-8.1, X6-2.1, X6-4.1, X6-6.1
Changed lines of the file:
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@@
 <part name="FRAME1" library="SparkFun-Aesthetics" deviceset="FRAME-A4L" device=""/>
 <part name="R1" library="rcl" deviceset="R-EU_" device="M1206"/>
+<part name="STEPPER-CTRL-X3" library="con-phoenix-508" deviceset="MSTBA6" device=""/>
+<part name="STEPPER-CTRL-X1" library="con-phoenix-508" deviceset="MSTBA6" device=""/>
+<part name="STEPPER-CTRL-Y" library="con-phoenix-508" deviceset="MSTBA6" device=""/>
+<part name="STEPPER-CTRL-Z" library="con-phoenix-508" deviceset="MSTBA6" device=""/>
+<part name="PWR-STEPPERS" library="con-phoenix-508" deviceset="MSTBA8" device=""/>
+<part name="X6" library="con-phoenix-508" deviceset="MSTBA6" device=""/>
+<part name="GND16" library="supply1" deviceset="GND" device=""/>
+<part name="GND17" library="supply1" deviceset="GND" device=""/>
 </parts>
 <sheets>
@@
 </plain>
 <instances>
+<instance part="PWR-STEPPERS" gate="-1" x="86.36" y="86.36"/>
+<instance part="PWR-STEPPERS" gate="-2" x="86.36" y="81.28"/>
+<instance part="PWR-STEPPERS" gate="-3" x="86.36" y="76.2"/>
+<instance part="PWR-STEPPERS" gate="-4" x="86.36" y="71.12"/>
+<instance part="PWR-STEPPERS" gate="-5" x="86.36" y="66.04"/>
+<instance part="PWR-STEPPERS" gate="-6" x="86.36" y="60.96"/>
+<instance part="PWR-STEPPERS" gate="-7" x="86.36" y="55.88"/>
+<instance part="PWR-STEPPERS" gate="-8" x="86.36" y="50.8"/>
+<instance part="X6" gate="-1" x="12.7" y="86.36"/>
+<instance part="X6" gate="-2" x="12.7" y="81.28"/>
+<instance part="X6" gate="-3" x="12.7" y="76.2"/>
+<instance part="X6" gate="-4" x="12.7" y="71.12"/>
+<instance part="X6" gate="-5" x="12.7" y="66.04"/>
+<instance part="X6" gate="-6" x="12.7" y="60.96"/>
+<instance part="GND16" gate="1" x="93.98" y="43.18"/>
+<instance part="GND17" gate="1" x="22.86" y="43.18"/>
 </instances>
 <busses>
+</busses>
+<nets>
+<net name="GND" class="0">
+<segment>
+<pinref part="GND17" gate="1" pin="GND"/>
+<wire x1="22.86" y1="45.72" x2="22.86" y2="60.96" width="0.1524" layer="91"/>
+<pinref part="X6" gate="-2" pin="1"/>
+<wire x1="22.86" y1="60.96" x2="22.86" y2="71.12" width="0.1524" layer="91"/>
+<wire x1="22.86" y1="71.12" x2="22.86" y2="81.28" width="0.1524" layer="91"/>
+<wire x1="22.86" y1="81.28" x2="17.78" y2="81.28" width="0.1524" layer="91"/>
+<pinref part="X6" gate="-4" pin="1"/>
+<wire x1="17.78" y1="71.12" x2="22.86" y2="71.12" width="0.1524" layer="91"/>
+<pinref part="X6" gate="-6" pin="1"/>
+<wire x1="17.78" y1="60.96" x2="22.86" y2="60.96" width="0.1524" layer="91"/>
+<junction x="22.86" y="60.96"/>
+<junction x="22.86" y="71.12"/>
+</segment>
+<segment>
+<pinref part="PWR-STEPPERS" gate="-8" pin="1"/>
+<wire x1="91.44" y1="50.8" x2="93.98" y2="50.8" width="0.1524" layer="91"/>
+<wire x1="93.98" y1="50.8" x2="93.98" y2="60.96" width="0.1524" layer="91"/>
+<pinref part="PWR-STEPPERS" gate="-6" pin="1"/>
+<wire x1="93.98" y1="60.96" x2="91.44" y2="60.96" width="0.1524" layer="91"/>
+<wire x1="93.98" y1="60.96" x2="93.98" y2="71.12" width="0.1524" layer="91"/>
+<pinref part="PWR-STEPPERS" gate="-4" pin="1"/>
+<wire x1="93.98" y1="71.12" x2="91.44" y2="71.12" width="0.1524" layer="91"/>
+<wire x1="93.98" y1="71.12" x2="93.98" y2="81.28" width="0.1524" layer="91"/>
+<pinref part="PWR-STEPPERS" gate="-2" pin="1"/>
+<wire x1="93.98" y1="81.28" x2="91.44" y2="81.28" width="0.1524" layer="91"/>
+<junction x="93.98" y="71.12"/>
+<junction x="93.98" y="60.96"/>
+<pinref part="GND16" gate="1" pin="GND"/>
+<wire x1="93.98" y1="45.72" x2="93.98" y2="50.8" width="0.1524" layer="91"/>
+<junction x="93.98" y="50.8"/>
+</segment>
+</net>
+<net name="+36V" class="0">
+<segment>
+<pinref part="X6" gate="-3" pin="1"/>
+<wire x1="17.78" y1="76.2" x2="33.02" y2="76.2" width="0.1524" layer="91"/>
+<label x="33.02" y="76.2" size="1.778" layer="95" xref="yes"/>
+</segment>
+<segment>
+<pinref part="PWR-STEPPERS" gate="-5" pin="1"/>
+<wire x1="91.44" y1="66.04" x2="99.06" y2="66.04" width="0.1524" layer="91"/>
+<pinref part="PWR-STEPPERS" gate="-3" pin="1"/>
+<wire x1="91.44" y1="76.2" x2="99.06" y2="76.2" width="0.1524" layer="91"/>
+<pinref part="PWR-STEPPERS" gate="-7" pin="1"/>
+<wire x1="99.06" y1="55.88" x2="91.44" y2="55.88" width="0.1524" layer="91"/>
+<wire x1="99.06" y1="55.88" x2="99.06" y2="66.04" width="0.1524" layer="91"/>
+<pinref part="PWR-STEPPERS" gate="-1" pin="1"/>
+<wire x1="99.06" y1="66.04" x2="99.06" y2="76.2" width="0.1524" layer="91"/>
+<wire x1="99.06" y1="76.2" x2="99.06" y2="86.36" width="0.1524" layer="91"/>
+<wire x1="91.44" y1="86.36" x2="99.06" y2="86.36" width="0.1524" layer="91"/>
+<junction x="99.06" y="66.04"/>
+<junction x="99.06" y="76.2"/>
+<junction x="99.06" y="86.36"/>
+<wire x1="99.06" y1="86.36" x2="109.22" y2="86.36" width="0.1524" layer="91"/>
+<label x="109.22" y="86.36" size="1.778" layer="95" xref="yes"/>
+</segment>
+</net>
+<net name="+48V" class="0">
+<segment>
+<pinref part="X6" gate="-5" pin="1"/>
+<wire x1="17.78" y1="66.04" x2="33.02" y2="66.04" width="0.1524" layer="91"/>
+<label x="33.02" y="66.04" size="1.778" layer="95" xref="yes"/>
+</segment>
+</net>
+<net name="+12V" class="0">
+<segment>
+<pinref part="X6" gate="-1" pin="1"/>
+<wire x1="17.78" y1="86.36" x2="33.02" y2="86.36" width="0.1524" layer="91"/>
+<label x="33.02" y="86.36" size="1.778" layer="95" xref="yes"/>
+</segment>
+</net>
+</nets>
+</sheet>
+<sheet>
+<description>Connectors</description>
+<plain>
+</plain>
+<instances>
+<instance part="STEPPER-CTRL-X3" gate="-1" x="66.04" y="93.98"/>
+<instance part="STEPPER-CTRL-X3" gate="-2" x="66.04" y="88.9"/>
+<instance part="STEPPER-CTRL-X3" gate="-3" x="66.04" y="83.82"/>
+<instance part="STEPPER-CTRL-X3" gate="-4" x="66.04" y="78.74"/>
+<instance part="STEPPER-CTRL-X3" gate="-5" x="66.04" y="73.66"/>
+<instance part="STEPPER-CTRL-X3" gate="-6" x="66.04" y="68.58"/>
+<instance part="STEPPER-CTRL-X1" gate="-1" x="66.04" y="60.96"/>
+<instance part="STEPPER-CTRL-X1" gate="-2" x="66.04" y="55.88"/>
+<instance part="STEPPER-CTRL-X1" gate="-3" x="66.04" y="50.8"/>
+<instance part="STEPPER-CTRL-X1" gate="-4" x="66.04" y="45.72"/>
+<instance part="STEPPER-CTRL-X1" gate="-5" x="66.04" y="40.64"/>
+<instance part="STEPPER-CTRL-X1" gate="-6" x="66.04" y="35.56"/>
+<instance part="STEPPER-CTRL-Y" gate="-1" x="66.04" y="27.94"/>
+<instance part="STEPPER-CTRL-Y" gate="-2" x="66.04" y="22.86"/>
+<instance part="STEPPER-CTRL-Y" gate="-3" x="66.04" y="17.78"/>
+<instance part="STEPPER-CTRL-Y" gate="-4" x="66.04" y="12.7"/>
+<instance part="STEPPER-CTRL-Y" gate="-5" x="66.04" y="7.62"/>
+<instance part="STEPPER-CTRL-Y" gate="-6" x="66.04" y="2.54"/>
+<instance part="STEPPER-CTRL-Z" gate="-1" x="66.04" y="-5.08"/>
+<instance part="STEPPER-CTRL-Z" gate="-2" x="66.04" y="-10.16"/>
+<instance part="STEPPER-CTRL-Z" gate="-3" x="66.04" y="-15.24"/>
+<instance part="STEPPER-CTRL-Z" gate="-4" x="66.04" y="-20.32"/>
+<instance part="STEPPER-CTRL-Z" gate="-5" x="66.04" y="-25.4"/>
+<instance part="STEPPER-CTRL-Z" gate="-6" x="66.04" y="-30.48"/>
+</instances>
+<busses>

Commit message: 20180427
Parts:
- removed C2: (no value), rcl:C-EU050-035X075
- removed PWR-STEPPERS: MSTBA8, con-phoenix-508:MSTBA8
- removed Q2: (no value), crystal:CRYSTALHC49S
- removed STEPPER-CTRL-X3, X6: MSTBA6, con-phoenix-508:MSTBA6
- added STEPPER-CTRL-X2: MSTBA6, con-phoenix-508:MSTBA6
Connections:
- removed net +36V: PWR-STEPPERS-1.1, PWR-STEPPERS-3.1, PWR-STEPPERS-5.1, PWR-STEPPERS-7.1, X6-3.1
- removed net +48V: X6-5.1
- net +12V: no longer X6-1.1
- net GND: no longer PWR-STEPPERS-2.1, PWR-STEPPERS-4.1, PWR-STEPPERS-6.1, PWR-STEPPERS-8.1, X6-2.1, X6-4.1, X6-6.1
- net MEGA2560.D0.RXD0: no longer C2.1
Changed lines of the file:
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@@
 <part name="GND7" library="supply1" deviceset="GND" device=""/>
 <part name="P+3" library="supply1" deviceset="+5V" device=""/>
-<part name="Q2" library="crystal" deviceset="CRYSTAL" device="HC49S"/>
-<part name="C2" library="rcl" deviceset="C-EU" device="050-035X075"/>
 <part name="JP.MEGA2560.POWER" library="pinhead" deviceset="PINHD-1X8" device=""/>
 <part name="JP.MEGA2560.ANALOG.LOW" library="pinhead" deviceset="PINHD-1X8" device=""/>
@@
 <part name="FRAME1" library="SparkFun-Aesthetics" deviceset="FRAME-A4L" device=""/>
 <part name="R1" library="rcl" deviceset="R-EU_" device="M1206"/>
-<part name="STEPPER-CTRL-X3" library="con-phoenix-508" deviceset="MSTBA6" device=""/>
+<part name="STEPPER-CTRL-X2" library="con-phoenix-508" deviceset="MSTBA6" device=""/>
 <part name="STEPPER-CTRL-X1" library="con-phoenix-508" deviceset="MSTBA6" device=""/>
 <part name="STEPPER-CTRL-Y" library="con-phoenix-508" deviceset="MSTBA6" device=""/>
 <part name="STEPPER-CTRL-Z" library="con-phoenix-508" deviceset="MSTBA6" device=""/>
-<part name="PWR-STEPPERS" library="con-phoenix-508" deviceset="MSTBA8" device=""/>
-<part name="X6" library="con-phoenix-508" deviceset="MSTBA6" device=""/>
-<part name="GND16" library="supply1" deviceset="GND" device=""/>
-<part name="GND17" library="supply1" deviceset="GND" device=""/>
 </parts>
 <sheets>
@@
 </plain>
 <instances>
-<instance part="Q2" gate="G$1" x="7.62" y="71.12"/>
-<instance part="C2" gate="G$1" x="35.56" y="66.04"/>
 </instances>
 <busses>
 </busses>
 <nets>
-<net name="MEGA2560.D0.RXD0" class="0">
-<segment>
-<pinref part="C2" gate="G$1" pin="1"/>
-<wire x1="35.56" y1="68.58" x2="35.56" y2="71.12" width="0.1524" layer="91"/>
-</segment>
-</net>
 </nets>
 </sheet>
@@
 </sheet>
 <sheet>
-<description>Питание</description>
-<plain>
-</plain>
-<instances>
-<instance part="PWR-STEPPERS" gate="-1" x="86.36" y="86.36"/>
-<instance part="PWR-STEPPERS" gate="-2" x="86.36" y="81.28"/>
-<instance part="PWR-STEPPERS" gate="-3" x="86.36" y="76.2"/>
-<instance part="PWR-STEPPERS" gate="-4" x="86.36" y="71.12"/>
-<instance part="PWR-STEPPERS" gate="-5" x="86.36" y="66.04"/>
-<instance part="PWR-STEPPERS" gate="-6" x="86.36" y="60.96"/>
-<instance part="PWR-STEPPERS" gate="-7" x="86.36" y="55.88"/>
-<instance part="PWR-STEPPERS" gate="-8" x="86.36" y="50.8"/>
-<instance part="X6" gate="-1" x="12.7" y="86.36"/>
-<instance part="X6" gate="-2" x="12.7" y="81.28"/>
-<instance part="X6" gate="-3" x="12.7" y="76.2"/>
-<instance part="X6" gate="-4" x="12.7" y="71.12"/>
-<instance part="X6" gate="-5" x="12.7" y="66.04"/>
-<instance part="X6" gate="-6" x="12.7" y="60.96"/>
-<instance part="GND16" gate="1" x="93.98" y="43.18"/>
-<instance part="GND17" gate="1" x="22.86" y="43.18"/>
-</instances>
-<busses>
-</busses>
-<nets>
-<net name="GND" class="0">
-<segment>
-<pinref part="GND17" gate="1" pin="GND"/>
-<wire x1="22.86" y1="45.72" x2="22.86" y2="60.96" width="0.1524" layer="91"/>
-<pinref part="X6" gate="-2" pin="1"/>
-<wire x1="22.86" y1="60.96" x2="22.86" y2="71.12" width="0.1524" layer="91"/>
-<wire x1="22.86" y1="71.12" x2="22.86" y2="81.28" width="0.1524" layer="91"/>
-<wire x1="22.86" y1="81.28" x2="17.78" y2="81.28" width="0.1524" layer="91"/>
-<pinref part="X6" gate="-4" pin="1"/>
-<wire x1="17.78" y1="71.12" x2="22.86" y2="71.12" width="0.1524" layer="91"/>
-<pinref part="X6" gate="-6" pin="1"/>
-<wire x1="17.78" y1="60.96" x2="22.86" y2="60.96" width="0.1524" layer="91"/>
-<junction x="22.86" y="60.96"/>
-<junction x="22.86" y="71.12"/>
-</segment>
-<segment>
-<pinref part="PWR-STEPPERS" gate="-8" pin="1"/>
-<wire x1="91.44" y1="50.8" x2="93.98" y2="50.8" width="0.1524" layer="91"/>
-<wire x1="93.98" y1="50.8" x2="93.98" y2="60.96" width="0.1524" layer="91"/>
-<pinref part="PWR-STEPPERS" gate="-6" pin="1"/>
-<wire x1="93.98" y1="60.96" x2="91.44" y2="60.96" width="0.1524" layer="91"/>
-<wire x1="93.98" y1="60.96" x2="93.98" y2="71.12" width="0.1524" layer="91"/>
-<pinref part="PWR-STEPPERS" gate="-4" pin="1"/>
-<wire x1="93.98" y1="71.12" x2="91.44" y2="71.12" width="0.1524" layer="91"/>
-<wire x1="93.98" y1="71.12" x2="93.98" y2="81.28" width="0.1524" layer="91"/>
-<pinref part="PWR-STEPPERS" gate="-2" pin="1"/>
-<wire x1="93.98" y1="81.28" x2="91.44" y2="81.28" width="0.1524" layer="91"/>
-<junction x="93.98" y="71.12"/>
-<junction x="93.98" y="60.96"/>
-<pinref part="GND16" gate="1" pin="GND"/>
-<wire x1="93.98" y1="45.72" x2="93.98" y2="50.8" width="0.1524" layer="91"/>
-<junction x="93.98" y="50.8"/>
-</segment>
-</net>
-<net name="+36V" class="0">
-<segment>
-<pinref part="X6" gate="-3" pin="1"/>
-<wire x1="17.78" y1="76.2" x2="33.02" y2="76.2" width="0.1524" layer="91"/>
-<label x="33.02" y="76.2" size="1.778" layer="95" xref="yes"/>
-</segment>
-<segment>
-<pinref part="PWR-STEPPERS" gate="-5" pin="1"/>
-<wire x1="91.44" y1="66.04" x2="99.06" y2="66.04" width="0.1524" layer="91"/>
-<pinref part="PWR-STEPPERS" gate="-3" pin="1"/>
-<wire x1="91.44" y1="76.2" x2="99.06" y2="76.2" width="0.1524" layer="91"/>
-<pinref part="PWR-STEPPERS" gate="-7" pin="1"/>
-<wire x1="99.06" y1="55.88" x2="91.44" y2="55.88" width="0.1524" layer="91"/>
-<wire x1="99.06" y1="55.88" x2="99.06" y2="66.04" width="0.1524" layer="91"/>
-<pinref part="PWR-STEPPERS" gate="-1" pin="1"/>
-<wire x1="99.06" y1="66.04" x2="99.06" y2="76.2" width="0.1524" layer="91"/>
-<wire x1="99.06" y1="76.2" x2="99.06" y2="86.36" width="0.1524" layer="91"/>
-<wire x1="91.44" y1="86.36" x2="99.06" y2="86.36" width="0.1524" layer="91"/>
-<junction x="99.06" y="66.04"/>
-<junction x="99.06" y="76.2"/>
-<junction x="99.06" y="86.36"/>
-<wire x1="99.06" y1="86.36" x2="109.22" y2="86.36" width="0.1524" layer="91"/>
-<label x="109.22" y="86.36" size="1.778" layer="95" xref="yes"/>
-</segment>
-</net>
-<net name="+48V" class="0">
-<segment>
-<pinref part="X6" gate="-5" pin="1"/>
-<wire x1="17.78" y1="66.04" x2="33.02" y2="66.04" width="0.1524" layer="91"/>
-<label x="33.02" y="66.04" size="1.778" layer="95" xref="yes"/>
-</segment>
-</net>
-<net name="+12V" class="0">
-<segment>
-<pinref part="X6" gate="-1" pin="1"/>
-<wire x1="17.78" y1="86.36" x2="33.02" y2="86.36" width="0.1524" layer="91"/>
-<label x="33.02" y="86.36" size="1.778" layer="95" xref="yes"/>
-</segment>
-</net>
-</nets>
-</sheet>
-<sheet>
 <description>Connectors</description>
 <plain>
 </plain>
 <instances>
-<instance part="STEPPER-CTRL-X3" gate="-1" x="66.04" y="93.98"/>
-<instance part="STEPPER-CTRL-X3" gate="-2" x="66.04" y="88.9"/>
-<instance part="STEPPER-CTRL-X3" gate="-3" x="66.04" y="83.82"/>
-<instance part="STEPPER-CTRL-X3" gate="-4" x="66.04" y="78.74"/>
-<instance part="STEPPER-CTRL-X3" gate="-5" x="66.04" y="73.66"/>
-<instance part="STEPPER-CTRL-X3" gate="-6" x="66.04" y="68.58"/>
+<instance part="STEPPER-CTRL-X2" gate="-1" x="66.04" y="93.98"/>
+<instance part="STEPPER-CTRL-X2" gate="-2" x="66.04" y="88.9"/>
+<instance part="STEPPER-CTRL-X2" gate="-3" x="66.04" y="83.82"/>
+<instance part="STEPPER-CTRL-X2" gate="-4" x="66.04" y="78.74"/>
+<instance part="STEPPER-CTRL-X2" gate="-5" x="66.04" y="73.66"/>
+<instance part="STEPPER-CTRL-X2" gate="-6" x="66.04" y="68.58"/>
 <instance part="STEPPER-CTRL-X1" gate="-1" x="66.04" y="60.96"/>
 <instance part="STEPPER-CTRL-X1" gate="-2" x="66.04" y="55.88"/>
