File: EAGLE/Control.Board/Control.Board.sch (EAGLE design)
At the start: 37 parts, among them J1 AVR_SPI_PROG_3X2PTH, U1.X LTV817LTV817S, U1.Y LTV817LTV817S, U1.Z LTV817LTV817S, U2.X LTV817LTV817S, U2.Y LTV817LTV817S, U2.Z LTV817LTV817S

Commit message: 20180503
Parts:
- added LED1, LED2, LED3, LED4: (no value), led:LEDCHIPLED_1206
- added R2, R3, R4, R5: (no value), rcl:R-EU_M1206
- added U$1, U$2, U$3, U$4: LTV817LTV817S, net173:LTV817LTV817S
- added X1: (no value), con-molex-micro-fit-3_0:HEADER_POS8_43045-0800
Connections:
- new net N$19: LED2.A, X1.8
- new net N$20: LED1.A, X1.6
- new net N$21: LED3.A, X1.4
- new net N$22: LED2.C, R4.1
- new net N$23: R4.2, U$1.A
- new net N$24: R5.2, U$2.A
- new net N$30: LED1.C, R5.1
- new net N$31: LED4.A, X1.2
- new net N$32: LED3.C, R3.1
- new net N$33: LED4.C, R2.1
- new net N$34: R2.2, U$4.A
- new net N$35: R3.2, U$3.A
- net +5V: now also X1.1, X1.3, X1.5, X1.7
- net GND: now also U$1.C, U$2.C, U$3.C, U$4.C
Changed lines of the file:
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@@
 <setting verticaltext="up"/>
 </settings>
-<grid distance="0.1" unitdist="inch" unit="inch" style="lines" multiple="1" display="no" altdistance="0.01" altunitdist="inch" altunit="inch"/>
+<grid distance="0.1" unitdist="inch" unit="inch" style="lines" multiple="1" display="yes" altdistance="0.01" altunitdist="inch" altunit="inch"/>
 <layers>
 <layer number="1" name="Top" color="4" fill="1" visible="no" active="no"/>
@@
 <part name="STEPPER-CTRL-Y" library="con-phoenix-508" deviceset="MSTBA6" device=""/>
 <part name="STEPPER-CTRL-Z" library="con-phoenix-508" deviceset="MSTBA6" device=""/>
+<part name="U$1" library="net173" deviceset="LTV817" device="LTV817S"/>
+<part name="U$2" library="net173" deviceset="LTV817" device="LTV817S"/>
+<part name="U$3" library="net173" deviceset="LTV817" device="LTV817S"/>
+<part name="U$4" library="net173" deviceset="LTV817" device="LTV817S"/>
+<part name="GND19" library="supply1" deviceset="GND" device=""/>
+<part name="R2" library="rcl" deviceset="R-EU_" device="M1206"/>
+<part name="R3" library="rcl" deviceset="R-EU_" device="M1206"/>
+<part name="R4" library="rcl" deviceset="R-EU_" device="M1206"/>
+<part name="R5" library="rcl" deviceset="R-EU_" device="M1206"/>
+<part name="LED1" library="led" deviceset="LED" device="CHIPLED_1206"/>
+<part name="LED2" library="led" deviceset="LED" device="CHIPLED_1206"/>
+<part name="LED3" library="led" deviceset="LED" device="CHIPLED_1206"/>
+<part name="LED4" library="led" deviceset="LED" device="CHIPLED_1206"/>
+<part name="X1" library="con-molex-micro-fit-3_0" deviceset="HEADER_POS8_?" device="43045-0800"/>
+<part name="P+7" library="supply1" deviceset="+5V" device=""/>
 </parts>
 <sheets>
@@
 </nets>
 </sheet>
+<sheet>
+<description>Buttons</description>
+<plain>
+<text x="40.64" y="-22.86" size="1.778" layer="91">Расчет обвязки оптрона PC817:
+VF(PC817) = 1.2 в
+VF(RED LED) = 1.9-2.3 в ≈ 2 в
+IF(RED LED) = 20 ma
+IF(PC817) = IF(RED LED) = 20 ma
+R = U/I = (12-1.2-2)/20 ma = 440Ω ≈ 470Ω
+CTR(PC817, 20 ma) = 125%</text>
+</plain>
+<instances>
+<instance part="U$1" gate="G$1" x="53.34" y="114.3"/>
+<instance part="U$2" gate="G$1" x="53.34" y="83.82"/>
+<instance part="U$3" gate="G$1" x="53.34" y="53.34"/>
+<instance part="U$4" gate="G$1" x="53.34" y="22.86"/>
+<instance part="GND19" gate="1" x="40.64" y="10.16"/>
+<instance part="R2" gate="G$1" x="30.48" y="25.4"/>
+<instance part="R3" gate="G$1" x="30.48" y="55.88"/>
+<instance part="R4" gate="G$1" x="30.48" y="116.84"/>
+<instance part="R5" gate="G$1" x="30.48" y="86.36"/>
+<instance part="LED1" gate="G$1" x="15.24" y="86.36" rot="R90"/>
+<instance part="LED2" gate="G$1" x="15.24" y="116.84" rot="R90"/>
+<instance part="LED3" gate="G$1" x="15.24" y="55.88" rot="R90"/>
+<instance part="LED4" gate="G$1" x="15.24" y="25.4" rot="R90"/>
+<instance part="X1" gate="G$1" x="-17.78" y="109.22" rot="R180"/>
+<instance part="P+7" gate="1" x="-7.62" y="124.46"/>
+</instances>
+<busses>
+</busses>
+<nets>
+<net name="GND" class="0">
+<segment>
+<pinref part="U$1" gate="G$1" pin="C"/>
+<pinref part="GND19" gate="1" pin="GND"/>
+<wire x1="43.18" y1="111.76" x2="40.64" y2="111.76" width="0.1524" layer="91"/>
+<wire x1="40.64" y1="111.76" x2="40.64" y2="81.28" width="0.1524" layer="91"/>
+<pinref part="U$4" gate="G$1" pin="C"/>
+<wire x1="40.64" y1="81.28" x2="40.64" y2="50.8" width="0.1524" layer="91"/>
+<wire x1="40.64" y1="50.8" x2="40.64" y2="20.32" width="0.1524" layer="91"/>
+<wire x1="40.64" y1="20.32" x2="40.64" y2="12.7" width="0.1524" layer="91"/>
+<wire x1="43.18" y1="20.32" x2="40.64" y2="20.32" width="0.1524" layer="91"/>
+<pinref part="U$3" gate="G$1" pin="C"/>
+<wire x1="43.18" y1="50.8" x2="40.64" y2="50.8" width="0.1524" layer="91"/>
+<pinref part="U$2" gate="G$1" pin="C"/>
+<wire x1="43.18" y1="81.28" x2="40.64" y2="81.28" width="0.1524" layer="91"/>
+<junction x="40.64" y="81.28"/>
+<junction x="40.64" y="50.8"/>
+<junction x="40.64" y="20.32"/>
+</segment>
+</net>
+<net name="+5V" class="0">
+<segment>
+<pinref part="P+7" gate="1" pin="+5V"/>
+<wire x1="-7.62" y1="121.92" x2="-7.62" y2="114.3" width="0.1524" layer="91"/>
+<pinref part="X1" gate="G$1" pin="1"/>
+<wire x1="-7.62" y1="114.3" x2="-7.62" y2="109.22" width="0.1524" layer="91"/>
+<wire x1="-7.62" y1="109.22" x2="-7.62" y2="104.14" width="0.1524" layer="91"/>
+<wire x1="-7.62" y1="104.14" x2="-7.62" y2="99.06" width="0.1524" layer="91"/>
+<wire x1="-7.62" y1="99.06" x2="-12.7" y2="99.06" width="0.1524" layer="91"/>
+<pinref part="X1" gate="G$1" pin="3"/>
+<wire x1="-12.7" y1="104.14" x2="-7.62" y2="104.14" width="0.1524" layer="91"/>
+<pinref part="X1" gate="G$1" pin="5"/>
+<wire x1="-12.7" y1="109.22" x2="-7.62" y2="109.22" width="0.1524" layer="91"/>
+<pinref part="X1" gate="G$1" pin="7"/>
+<wire x1="-12.7" y1="114.3" x2="-7.62" y2="114.3" width="0.1524" layer="91"/>
+<junction x="-7.62" y="114.3"/>
+<junction x="-7.62" y="109.22"/>
+<junction x="-7.62" y="104.14"/>
+</segment>
+</net>
+<net name="N$19" class="0">
+<segment>
+<pinref part="X1" gate="G$1" pin="8"/>
+<pinref part="LED2" gate="G$1" pin="A"/>
+<wire x1="-12.7" y1="116.84" x2="12.7" y2="116.84" width="0.1524" layer="91"/>
+</segment>
+</net>
+<net name="N$20" class="0">
+<segment>
+<pinref part="X1" gate="G$1" pin="6"/>
+<wire x1="-12.7" y1="111.76" x2="10.16" y2="111.76" width="0.1524" layer="91"/>
+<wire x1="10.16" y1="111.76" x2="10.16" y2="86.36" width="0.1524" layer="91"/>
+<pinref part="LED1" gate="G$1" pin="A"/>
+<wire x1="10.16" y1="86.36" x2="12.7" y2="86.36" width="0.1524" layer="91"/>
+</segment>
+</net>
+<net name="N$21" class="0">
+<segment>
+<pinref part="X1" gate="G$1" pin="4"/>
+<wire x1="-12.7" y1="106.68" x2="5.08" y2="106.68" width="0.1524" layer="91"/>
+<wire x1="5.08" y1="106.68" x2="5.08" y2="55.88" width="0.1524" layer="91"/>
+<pinref part="LED3" gate="G$1" pin="A"/>
+<wire x1="5.08" y1="55.88" x2="12.7" y2="55.88" width="0.1524" layer="91"/>
+</segment>
+</net>
+<net name="N$22" class="0">
+<segment>
+<pinref part="LED2" gate="G$1" pin="C"/>
+<pinref part="R4" gate="G$1" pin="1"/>
+<wire x1="20.32" y1="116.84" x2="25.4" y2="116.84" width="0.1524" layer="91"/>
+</segment>
+</net>
+<net name="N$23" class="0">
+<segment>
+<pinref part="R4" gate="G$1" pin="2"/>
+<pinref part="U$1" gate="G$1" pin="A"/>
+<wire x1="35.56" y1="116.84" x2="43.18" y2="116.84" width="0.1524" layer="91"/>
+</segment>
+</net>
+<net name="N$24" class="0">
+<segment>
+<pinref part="R5" gate="G$1" pin="2"/>
+<pinref part="U$2" gate="G$1" pin="A"/>
+<wire x1="35.56" y1="86.36" x2="43.18" y2="86.36" width="0.1524" layer="91"/>
+</segment>
+</net>
+<net name="N$30" class="0">
+<segment>
+<pinref part="LED1" gate="G$1" pin="C"/>
+<pinref part="R5" gate="G$1" pin="1"/>
+<wire x1="20.32" y1="86.36" x2="25.4" y2="86.36" width="0.1524" layer="91"/>
+</segment>
+</net>
+<net name="N$31" class="0">
+<segment>
+<pinref part="LED4" gate="G$1" pin="A"/>
+<wire x1="12.7" y1="25.4" x2="0" y2="25.4" width="0.1524" layer="91"/>
+<wire x1="0" y1="25.4" x2="0" y2="101.6" width="0.1524" layer="91"/>
+<pinref part="X1" gate="G$1" pin="2"/>
+<wire x1="0" y1="101.6" x2="-12.7" y2="101.6" width="0.1524" layer="91"/>
+</segment>
+</net>
+<net name="N$32" class="0">
+<segment>
+<pinref part="LED3" gate="G$1" pin="C"/>
+<pinref part="R3" gate="G$1" pin="1"/>
+<wire x1="20.32" y1="55.88" x2="25.4" y2="55.88" width="0.1524" layer="91"/>
+</segment>
+</net>
+<net name="N$33" class="0">
+<segment>
+<pinref part="LED4" gate="G$1" pin="C"/>
+<pinref part="R2" gate="G$1" pin="1"/>
+<wire x1="20.32" y1="25.4" x2="25.4" y2="25.4" width="0.1524" layer="91"/>
+</segment>
+</net>
+<net name="N$34" class="0">
+<segment>
+<pinref part="R2" gate="G$1" pin="2"/>
+<pinref part="U$4" gate="G$1" pin="A"/>
+<wire x1="35.56" y1="25.4" x2="43.18" y2="25.4" width="0.1524" layer="91"/>
+</segment>
+</net>
+<net name="N$35" class="0">
+<segment>
+<pinref part="R3" gate="G$1" pin="2"/>
+<pinref part="U$3" gate="G$1" pin="A"/>
+<wire x1="35.56" y1="55.88" x2="43.18" y2="55.88" width="0.1524" layer="91"/>
+</segment>
+</net>
+</nets>
+</sheet>

Commit message: 20180503
Parts:
- removed STEPPER-CTRL-X1, STEPPER-CTRL-X2, STEPPER-CTRL-Y, STEPPER-CTRL-Z: MSTBA6, con-phoenix-508:MSTBA6
- added STEPPER-X1, STEPPER-X2, STEPPER-Y, STEPPER-Z: (no value), con-molex-micro-fit-3_0:HEADER_POS6_43045-0600
- R2, R3, R4, R5: value (none) -> 100
Connections:
- net +5V: now also STEPPER-X1.1, STEPPER-X1.2, STEPPER-X1.3, STEPPER-X2.1, STEPPER-X2.2, STEPPER-X2.3, STEPPER-Y.1, STEPPER-Y.2, STEPPER-Y.3, STEPPER-Z.1, STEPPER-Z.2, STEPPER-Z.3, X1.2, X1.4; no longer X1.5, X1.7
- net GND: now also U$1.EMIT, U$2.EMIT, U$3.EMIT, U$4.EMIT
- net MEGA2560.A10.CYCLE.START: now also U$3.COL
- net MEGA2560.A11.SAFETY.DOOR: now also U$4.COL
- net MEGA2560.A8.RESET.ABORT: now also U$1.COL
- net MEGA2560.A9.FEED.HOLD: now also U$2.COL
- net MEGA2560.D13.STEPPER.EN: now also STEPPER-X1.6, STEPPER-X2.6, STEPPER-Y.6, STEPPER-Z.6
- net MEGA2560.D24.STEP.X: now also STEPPER-X1.4, STEPPER-X2.4
- net MEGA2560.D25.STEP.Y: now also STEPPER-Y.4
- net MEGA2560.D26.STEP.Z: now also STEPPER-Z.4
- net MEGA2560.D30.DIR.X: now also STEPPER-X1.5, STEPPER-X2.5
- net MEGA2560.D31.DIR.Y: now also STEPPER-Y.5
- net MEGA2560.D32.DIR.Z: now also STEPPER-Z.5
- net N$20: now also X1.7; no longer X1.6
- net N$21: now also X1.6; no longer X1.4
- net N$31: now also X1.5; no longer X1.2
Other:
- note added: "Расчет обвязки оптрона PC817: VF(PC817) = 1.2 в VF(RED LED) = 1.8-2.0 в ≈ 2 в IF(RED LED) = 20 ma IF(PC817) = IF(RED LED) = 20 ma R = U/I = (5-1.2-2)/20 ma = 90Ω ≈ 100Ω CTR(PC817, 20 ma) = 125% 1206 Red 100-120 1.8-2.0V 20MA 1206 Blue 120-150 3.0-3.2V 20MA 1206 Green 400-500 3.0-3.2V 20MA 1206 Yellow 120-150 1.8-2.0V 20MA 1206 White 500-600 3.0-3.2V 20MA"
