File: EAGLE/!PRJ/Probe.Board/Probe.Board.sch (EAGLE design)
At the start: 0 parts

Commit message: 20180504
Parts:
- added LED, PROBE-IN, PROBE-OUT: (no value), pinhead:PINHD-1X2/90
- added OK1: PC817, optocoupler:PC817
- added R1: 100, rcl:R-EU_0207/12
- added U1: TSP-05TSP-05, net173:TSP-05TSP-05
- added X1: MSTBA2, con-phoenix-508:MSTBA2
Connections:
- new net GND: OK1.C, U1.VOUT-
- new net N$1: U1.AC2, X1-2.1
- new net N$2: U1.AC1, X1-1.1
- new net N$3: OK1.EMIT, PROBE-OUT.2
- new net N$4: OK1.COL, PROBE-OUT.1
- new net N$5: OK1.A, R1.1
- new net N$6: LED.2, R1.2
- new net N$7: LED.1, PROBE-IN.2
- new net N$8: PROBE-IN.1, U1.VOUT+
Other:
- note added: "Расчет обвязки оптрона PC817: VF(PC817) = 1.2 в VF(RED LED) = 1.9-2.1 в ≈ 2 в IF(RED LED) = 20 ma IF(PC817) = IF(RED LED) = 20 ma R = U/I = (5-1.2-2)/20 ma = 90Ω ≈ 100Ω CTR(PC817, 20 ma) = 125%"
Changed lines of the file:
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@@
 <grid distance="0.1" unitdist="inch" unit="inch" style="lines" multiple="1" display="no" altdistance="0.01" altunitdist="inch" altunit="inch"/>
 <layers>
+<layer number="1" name="Top" color="4" fill="1" visible="no" active="no"/>
+<layer number="2" name="Route2" color="1" fill="3" visible="no" active="no"/>
+<layer number="3" name="Route3" color="4" fill="3" visible="no" active="no"/>
+<layer number="4" name="Route4" color="1" fill="4" visible="no" active="no"/>
+<layer number="5" name="Route5" color="4" fill="4" visible="no" active="no"/>
+<layer number="6" name="Route6" color="1" fill="8" visible="no" active="no"/>
+<layer number="7" name="Route7" color="4" fill="8" visible="no" active="no"/>
+<layer number="8" name="Route8" color="1" fill="2" visible="no" active="no"/>
+<layer number="9" name="Route9" color="4" fill="2" visible="no" active="no"/>
+<layer number="10" name="Route10" color="1" fill="7" visible="no" active="no"/>
+<layer number="11" name="Route11" color="4" fill="7" visible="no" active="no"/>
+<layer number="12" name="Route12" color="1" fill="5" visible="no" active="no"/>
+<layer number="13" name="Route13" color="4" fill="5" visible="no" active="no"/>
+<layer number="14" name="Route14" color="1" fill="6" visible="no" active="no"/>
+<layer number="15" name="Route15" color="4" fill="6" visible="no" active="no"/>
+<layer number="16" name="Bottom" color="1" fill="1" visible="no" active="no"/>
+<layer number="17" name="Pads" color="2" fill="1" visible="no" active="no"/>
+<layer number="18" name="Vias" color="2" fill="1" visible="no" active="no"/>
+<layer number="19" name="Unrouted" color="6" fill="1" visible="no" active="no"/>
+<layer number="20" name="Dimension" color="15" fill="1" visible="no" active="no"/>
+<layer number="21" name="tPlace" color="7" fill="1" visible="no" active="no"/>
+<layer number="22" name="bPlace" color="7" fill="1" visible="no" active="no"/>
+<layer number="23" name="tOrigins" color="15" fill="1" visible="no" active="no"/>
+<layer number="24" name="bOrigins" color="15" fill="1" visible="no" active="no"/>
+<layer number="25" name="tNames" color="7" fill="1" visible="no" active="no"/>
+<layer number="26" name="bNames" color="7" fill="1" visible="no" active="no"/>
+<layer number="27" name="tValues" color="7" fill="1" visible="no" active="no"/>
+<layer number="28" name="bValues" color="7" fill="1" visible="no" active="no"/>
+<layer number="29" name="tStop" color="7" fill="3" visible="no" active="no"/>
+<layer number="30" name="bStop" color="7" fill="6" visible="no" active="no"/>
+<layer number="31" name="tCream" color="7" fill="4" visible="no" active="no"/>
+<layer number="32" name="bCream" color="7" fill="5" visible="no" active="no"/>
+<layer number="33" name="tFinish" color="6" fill="3" visible="no" active="no"/>
+<layer number="34" name="bFinish" color="6" fill="6" visible="no" active="no"/>
+<layer number="35" name="tGlue" color="7" fill="4" visible="no" active="no"/>
+<layer number="36" name="bGlue" color="7" fill="5" visible="no" active="no"/>
+<layer number="37" name="tTest" color="7" fill="1" visible="no" active="no"/>
+<layer number="38" name="bTest" color="7" fill="1" visible="no" active="no"/>
+<layer number="39" name="tKeepout" color="4" fill="11" visible="no" active="no"/>
+<layer number="40" name="bKeepout" color="1" fill="11" visible="no" active="no"/>
+<layer number="41" name="tRestrict" color="4" fill="10" visible="no" active="no"/>
+<layer number="42" name="bRestrict" color="1" fill="10" visible="no" active="no"/>
+<layer number="43" name="vRestrict" color="2" fill="10" visible="no" active="no"/>
+<layer number="44" name="Drills" color="7" fill="1" visible="no" active="no"/>
+<layer number="45" name="Holes" color="7" fill="1" visible="no" active="no"/>
+<layer number="46" name="Milling" color="3" fill="1" visible="no" active="no"/>
+<layer number="47" name="Measures" color="7" fill="1" visible="no" active="no"/>
+<layer number="48" name="Document" color="7" fill="1" visible="no" active="no"/>
+<layer number="49" name="Reference" color="7" fill="1" visible="no" active="no"/>
+<layer number="51" name="tDocu" color="7" fill="1" visible="no" active="no"/>
+<layer number="52" name="bDocu" color="7" fill="1" visible="no" active="no"/>
 <layer number="91" name="Nets" color="2" fill="1" visible="yes" active="yes"/>
 <layer number="92" name="Busses" color="1" fill="1" visible="yes" active="yes"/>
@@
 </classes>
 <parts>
+<part name="PROBE-IN" library="pinhead" deviceset="PINHD-1X2" device="/90"/>
+<part name="PROBE-OUT" library="pinhead" deviceset="PINHD-1X2" device="/90"/>
+<part name="OK1" library="optocoupler" deviceset="PC817" device=""/>
+<part name="X1" library="con-phoenix-508" deviceset="MSTBA2" device=""/>
+<part name="GND1" library="supply1" deviceset="GND" device=""/>
+<part name="R1" library="rcl" deviceset="R-EU_" device="0207/12" value="100"/>
+<part name="LED" library="pinhead" deviceset="PINHD-1X2" device="/90"/>
+<part name="U1" library="net173" deviceset="TSP-05" device="TSP-05"/>
+<part name="GND2" library="supply1" deviceset="GND" device=""/>
 </parts>
 <sheets>
 <sheet>
 <plain>
+<text x="-10.16" y="71.12" size="1.778" layer="91">Расчет обвязки оптрона PC817:
+VF(PC817) = 1.2 в
+VF(RED LED) = 1.9-2.1 в ≈ 2 в
+IF(RED LED) = 20 ma
+IF(PC817) = IF(RED LED) = 20 ma
+R = U/I = (5-1.2-2)/20 ma = 90Ω ≈ 100Ω
+CTR(PC817, 20 ma) = 125%</text>
 </plain>
 <instances>
+<instance part="PROBE-IN" gate="G$1" x="68.58" y="83.82" rot="R90"/>
+<instance part="PROBE-OUT" gate="G$1" x="144.78" y="43.18"/>
+<instance part="OK1" gate="A" x="96.52" y="45.72"/>
+<instance part="X1" gate="-1" x="0" y="48.26"/>
+<instance part="X1" gate="-2" x="0" y="43.18"/>
+<instance part="GND1" gate="1" x="81.28" y="35.56"/>
+<instance part="R1" gate="G$1" x="81.28" y="58.42" rot="R90"/>
+<instance part="LED" gate="G$1" x="81.28" y="83.82" rot="R90"/>
+<instance part="U1" gate="G$1" x="33.02" y="48.26"/>
+<instance part="GND2" gate="1" x="58.42" y="50.8"/>
 </instances>
 <busses>
 </busses>
 <nets>
+<net name="GND" class="0">
+<segment>
+<pinref part="OK1" gate="A" pin="C"/>
+<pinref part="GND1" gate="1" pin="GND"/>
+<wire x1="81.28" y1="43.18" x2="86.36" y2="43.18" width="0.1524" layer="91"/>
+<wire x1="81.28" y1="43.18" x2="81.28" y2="38.1" width="0.1524" layer="91"/>
+</segment>
+<segment>
+<pinref part="U1" gate="G$1" pin="VOUT-"/>
+<pinref part="GND2" gate="1" pin="GND"/>
+<wire x1="55.88" y1="55.88" x2="58.42" y2="55.88" width="0.1524" layer="91"/>
+<wire x1="58.42" y1="55.88" x2="58.42" y2="53.34" width="0.1524" layer="91"/>
+</segment>
+</net>
+<net name="N$3" class="0">
+<segment>
+<pinref part="OK1" gate="A" pin="EMIT"/>
+<pinref part="PROBE-OUT" gate="G$1" pin="2"/>
+<wire x1="104.14" y1="43.18" x2="142.24" y2="43.18" width="0.1524" layer="91"/>
+</segment>
+</net>
+<net name="N$4" class="0">
+<segment>
+<pinref part="OK1" gate="A" pin="COL"/>
+<wire x1="104.14" y1="48.26" x2="121.92" y2="48.26" width="0.1524" layer="91"/>
+<wire x1="121.92" y1="48.26" x2="121.92" y2="45.72" width="0.1524" layer="91"/>
+<pinref part="PROBE-OUT" gate="G$1" pin="1"/>
+<wire x1="121.92" y1="45.72" x2="142.24" y2="45.72" width="0.1524" layer="91"/>
+</segment>
+</net>
+<net name="N$5" class="0">
+<segment>
+<pinref part="OK1" gate="A" pin="A"/>
+<pinref part="R1" gate="G$1" pin="1"/>
+<wire x1="86.36" y1="48.26" x2="81.28" y2="48.26" width="0.1524" layer="91"/>
+<wire x1="81.28" y1="48.26" x2="81.28" y2="53.34" width="0.1524" layer="91"/>
+</segment>
+</net>
+<net name="N$6" class="0">
+<segment>
+<pinref part="R1" gate="G$1" pin="2"/>
+<pinref part="LED" gate="G$1" pin="2"/>
+<wire x1="81.28" y1="63.5" x2="81.28" y2="81.28" width="0.1524" layer="91"/>
+</segment>
+</net>
+<net name="N$7" class="0">
+<segment>
+<pinref part="LED" gate="G$1" pin="1"/>
+<wire x1="78.74" y1="81.28" x2="78.74" y2="73.66" width="0.1524" layer="91"/>
+<pinref part="PROBE-IN" gate="G$1" pin="2"/>
+<wire x1="78.74" y1="73.66" x2="68.58" y2="73.66" width="0.1524" layer="91"/>
+<wire x1="68.58" y1="73.66" x2="68.58" y2="81.28" width="0.1524" layer="91"/>
+</segment>
+</net>
+<net name="N$8" class="0">
+<segment>
+<pinref part="PROBE-IN" gate="G$1" pin="1"/>
+<wire x1="66.04" y1="81.28" x2="66.04" y2="40.64" width="0.1524" layer="91"/>
+<pinref part="U1" gate="G$1" pin="VOUT+"/>
+<wire x1="55.88" y1="40.64" x2="66.04" y2="40.64" width="0.1524" layer="91"/>
+</segment>
+</net>
+<net name="N$1" class="0">
+<segment>
+<pinref part="X1" gate="-2" pin="1"/>
+<pinref part="U1" gate="G$1" pin="AC2"/>
+<wire x1="5.08" y1="43.18" x2="10.16" y2="43.18" width="0.1524" layer="91"/>
+</segment>
+</net>
+<net name="N$2" class="0">
+<segment>
+<pinref part="X1" gate="-1" pin="1"/>
+<wire x1="5.08" y1="48.26" x2="7.62" y2="48.26" width="0.1524" layer="91"/>
+<wire x1="7.62" y1="48.26" x2="7.62" y2="53.34" width="0.1524" layer="91"/>
+<pinref part="U1" gate="G$1" pin="AC1"/>
+<wire x1="7.62" y1="53.34" x2="10.16" y2="53.34" width="0.1524" layer="91"/>
+</segment>
+</net>
 </nets>
 </sheet>
@@
 </schematic>
 </drawing>
+<compatibility>
+<note version="6.3" minversion="6.2.2" severity="warning">
+Since Version 6.2.2 text objects can contain more than one line,
+which will not be processed correctly with this version.
+</note>
+</compatibility>
 </eagle>
