File: EAGLE/!PRJ/Control.Board/Control.Board.brd (EAGLE design)
At the start: 160 x 100 mm, 50 parts, among them J1 AVR_SPI_PROG_3X2PTH, U1.X LTV817LTV817S, U1.Y LTV817LTV817S, U1.Z LTV817LTV817S, U2.X LTV817LTV817S, U2.Y LTV817LTV817S, U2.Z LTV817LTV817S

Commit message: 20180505
Parts:
- removed JP.LIMIT.X, JP.LIMIT.Y, JP.LIMIT.Z: (no value), pinhead:1X06
- removed LED1.X, LED1.Y, LED1.Z, LED2.X, LED2.Y, LED2.Z: (no value), led:CHIPLED_0805
- removed R1: (no value), rcl:M1206
- removed R1.X, R1.Y, R1.Z, R2.X, R2.Y, R2.Z: 470, rcl:M0805
- removed R3.X, R3.Y, R3.Z: 10K, rcl:M0805
- added EXT.JP: (no value), pinhead:2X11/90
- added JP1: (no value), pinhead:2X09/90
- added LED.X.1, LED.X.2, LED.Y.1, LED.Y.2, LED.Z.1, LED.Z.2: (no value), led:CHIPLED_1206
- added PROBE: (no value), pinhead:1X02/90
- added PWR.JP: (no value), pinhead:1X03/90
- added R.X.1, R.X.2, R.Y.1, R.Y.2, R.Z.1, R.Z.2: 470, rcl:M1206
Connections:
- removed net N$13: JP.LIMIT.Z.2, R1.Z.1
- removed net N$15: JP.LIMIT.Z.5, R2.Z.1
- removed net N$2: JP.LIMIT.Y.2, R1.Y.1
- removed net N$4: JP.LIMIT.X.2, R1.X.1
- removed net N$6: JP.LIMIT.X.5, R2.X.1
- removed net N$9: JP.LIMIT.Y.5, R2.Y.1
- new net SENSOR.LIMIT.X.1: JP1.3, R.X.1.1
- new net SENSOR.LIMIT.X.2: JP1.4, R.X.2.1
- new net SENSOR.LIMIT.Y.1: JP1.9, R.Y.1.1
- new net SENSOR.LIMIT.Y.2: JP1.10, R.Y.2.1
- new net SENSOR.LIMIT.Z.1: JP1.15, R.Z.1.1
- new net SENSOR.LIMIT.Z.2: JP1.16, R.Z.2.1
- net +12V: now also EXT.JP.1, EXT.JP.2, EXT.JP.7, EXT.JP.8, JP1.1, JP1.13, JP1.14, JP1.2, JP1.7, JP1.8, PWR.JP.1; no longer JP.LIMIT.X.1, JP.LIMIT.X.4, JP.LIMIT.Y.1, JP.LIMIT.Y.4, JP.LIMIT.Z.1, JP.LIMIT.Z.4
- net +5V: now also EXT.JP.10, EXT.JP.3, EXT.JP.4, EXT.JP.9, PWR.JP.2; no longer R3.X.2, R3.Y.2, R3.Z.2
- net GND: now also EXT.JP.11, EXT.JP.12, EXT.JP.5, EXT.JP.6, JP1.11, JP1.12, JP1.17, JP1.18, JP1.5, JP1.6, PROBE.2, PWR.JP.3; no longer JP.LIMIT.X.3, JP.LIMIT.X.6, JP.LIMIT.Y.3, JP.LIMIT.Y.6, JP.LIMIT.Z.3, JP.LIMIT.Z.6
- net MEGA2560.A15.PROBE: now also PROBE.1
- net MEGA2560.D0.RXD0: now also EXT.JP.21, EXT.JP.22
- net MEGA2560.D1.TXD0: now also EXT.JP.19, EXT.JP.20
- net MEGA2560.D10.LIMIT.X: now also EXT.JP.13, EXT.JP.14; no longer R3.X.1
- net MEGA2560.D11.LIMIT.Y: now also EXT.JP.15, EXT.JP.16; no longer R3.Y.1
- net MEGA2560.D12.LIMIT.Z: now also EXT.JP.17, EXT.JP.18; no longer R3.Z.1
- net N$1: now also LED.X.2.C; no longer LED2.X.C
- net N$10: now also LED.Y.2.A, R.Y.2.2; no longer LED2.Y.A, R2.Y.2
- net N$11: now also LED.Y.2.C; no longer LED2.Y.C
- net N$12: now also LED.Y.1.C; no longer LED1.Y.C
- net N$14: now also LED.Z.1.A, R.Z.1.2; no longer LED1.Z.A, R1.Z.2
- net N$16: now also LED.Z.2.A, R.Z.2.2; no longer LED2.Z.A, R2.Z.2
- net N$17: now also LED.Z.2.C; no longer LED2.Z.C
- net N$18: now also LED.Z.1.C; no longer LED1.Z.C
- net N$3: now also LED.Y.1.A, R.Y.1.2; no longer LED1.Y.A, R1.Y.2
- net N$5: now also LED.X.1.A, R.X.1.2; no longer LED1.X.A, R1.X.2
- net N$7: now also LED.X.2.A, R.X.2.2; no longer LED2.X.A, R2.X.2
- net N$8: now also LED.X.1.C; no longer LED1.X.C

Commit message: 20180510
Parts:
- added COOLANT.JP: (no value), pinhead:1X04/90
- added LED5, LED6: (no value), led:CHIPLED_1206
- added R1, R6: 100, rcl:M1206
- added U$5, U$6: LTV817LTV817S, net173:DIL4-SMD
- added X2: (no value), con-molex-micro-fit-3_0:43045-0400
Connections:
- new net N$13: COOLANT.JP.1, U$5.4
- new net N$15: COOLANT.JP.3, U$6.4
- new net N$2: R1.2, U$5.1
- new net N$36: LED6.C, R6.1
- new net N$37: R6.2, U$6.1
- new net N$4: LED5.C, R1.1
- new net N$6: COOLANT.JP.2, U$5.3
- new net N$9: COOLANT.JP.4, U$6.3
- net GND: now also U$5.2, U$6.2, X2.P$4
- net MEGA2560.D5.SPINDLE.DIR: now also X2.P$3
- net MEGA2560.D6.SPINDLE.EN: now also X2.P$2
- net MEGA2560.D7.SPINDLE.PWM: now also X2.P$1
- net MEGA2560.D8.COOLANT.FLOOD: now also LED5.A
- net MEGA2560.D9.COOLANT.MIST: now also LED6.A
Changed lines of the file:
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@@
 <element name="EXT.JP" library="pinhead" package="2X11/90" value="" x="-124.46" y="-370.84"/>
 <element name="PWR.JP" library="pinhead" package="1X03/90" value="" x="-148.59" y="-372.11"/>
+<element name="R1" library="rcl" package="M1206" value="100" x="-151.13" y="-382.27"/>
+<element name="LED5" library="led" package="CHIPLED_1206" value="" x="-158.75" y="-381"/>
+<element name="U$5" library="net173" package="DIL4-SMD" value="LTV817LTV817S" x="-166.37" y="-377.19"/>
+<element name="U$6" library="net173" package="DIL4-SMD" value="LTV817LTV817S" x="-175.26" y="-377.19"/>
+<element name="COOLANT.JP" library="pinhead" package="1X04/90" value="" x="-171.45" y="-391.16"/>
+<element name="R6" library="rcl" package="M1206" value="100" x="-176.53" y="-400.05"/>
+<element name="LED6" library="led" package="CHIPLED_1206" value="" x="-182.88" y="-398.78"/>
+<element name="X2" library="con-molex-micro-fit-3_0" package="43045-0400" value="" x="-191.77" y="-397.51">
+<attribute name="MATERIAL" value="" x="-191.77" y="-397.51" size="1.778" layer="27" display="off"/>
+</element>
 </elements>
 <signals>
@@
 <contactref element="EXT.JP" pad="11"/>
 <contactref element="PWR.JP" pad="3"/>
+<contactref element="U$5" pad="2"/>
+<contactref element="U$6" pad="2"/>
+<contactref element="X2" pad="P$4"/>
 <wire x1="-132.08" y1="-377.19" x2="-132.08" y2="-374.65" width="0" layer="19" extent="1-1"/>
 <wire x1="-124.46" y1="-377.19" x2="-132.08" y2="-377.19" width="0" layer="19" extent="1-1"/>
 <wire x1="-124.46" y1="-374.65" x2="-124.46" y2="-377.19" width="0" layer="19" extent="1-1"/>
 <wire x1="-146.05" y1="-375.92" x2="-132.08" y2="-374.65" width="0" layer="19" extent="1-1"/>
+<wire x1="-165.1" y1="-381.96" x2="-146.05" y2="-375.92" width="0" layer="19" extent="1-1"/>
+<wire x1="-173.99" y1="-381.96" x2="-165.1" y2="-381.96" width="0" layer="19" extent="1-1"/>
+<wire x1="-193.27" y1="-390.19" x2="-173.99" y2="-381.96" width="0" layer="19" extent="1-1"/>
 <wire x1="-93.98" y1="-322.58" x2="-124.46" y2="-374.65" width="0" layer="19" extent="1-1"/>
 <wire x1="-93.98" y1="-320.04" x2="-93.98" y2="-322.58" width="0" layer="19" extent="1-1"/>
@@
 <signal name="MEGA2560.D5.SPINDLE.DIR">
 <contactref element="JP.MEGA2560.PWM.LOW" pad="3"/>
+<contactref element="X2" pad="P$3"/>
+<wire x1="-190.27" y1="-390.19" x2="53.34" y2="55.88" width="0" layer="19" extent="1-1"/>
 </signal>
 <signal name="MEGA2560.D6.SPINDLE.EN">
 <contactref element="JP.MEGA2560.PWM.LOW" pad="2"/>
+<contactref element="X2" pad="P$2"/>
+<wire x1="-193.27" y1="-393.19" x2="53.34" y2="58.42" width="0" layer="19" extent="1-1"/>
 </signal>
 <signal name="MEGA2560.D7.SPINDLE.PWM">
 <contactref element="JP.MEGA2560.PWM.LOW" pad="1"/>
+<contactref element="X2" pad="P$1"/>
+<wire x1="-190.27" y1="-393.19" x2="53.34" y2="60.96" width="0" layer="19" extent="1-1"/>
 </signal>
 <signal name="MEGA2560.D8.COOLANT.FLOOD">
 <contactref element="JP.MEGA2560.PWM.HIGH" pad="10"/>
+<contactref element="LED5" pad="A"/>
+<wire x1="-158.75" y1="-382.75" x2="53.34" y2="64.77" width="0" layer="19" extent="1-1"/>
 </signal>
 <signal name="MEGA2560.D9.COOLANT.MIST">
 <contactref element="JP.MEGA2560.PWM.HIGH" pad="9"/>
+<contactref element="LED6" pad="A"/>
+<wire x1="-182.88" y1="-400.53" x2="53.34" y2="67.31" width="0" layer="19" extent="1-1"/>
 </signal>
 <signal name="MEGA2560.D10.LIMIT.X">
@@
 <wire x1="-130.68" y1="-359.41" x2="-138.43" y2="-361.16" width="0" layer="19" extent="1-1"/>
 </signal>
+<signal name="N$2">
+<contactref element="U$5" pad="1"/>
+<contactref element="R1" pad="2"/>
+<wire x1="-149.73" y1="-382.27" x2="-167.64" y2="-381.96" width="0" layer="19" extent="1-1"/>
+</signal>
+<signal name="N$4">
+<contactref element="R1" pad="1"/>
+<contactref element="LED5" pad="C"/>
+<wire x1="-152.53" y1="-382.27" x2="-158.75" y2="-379.25" width="0" layer="19" extent="1-1"/>
+</signal>
+<signal name="N$6">
+<contactref element="U$5" pad="3"/>
+<contactref element="COOLANT.JP" pad="2"/>
+<wire x1="-165.1" y1="-372.42" x2="-172.72" y2="-394.97" width="0" layer="19" extent="1-1"/>
+</signal>
+<signal name="N$9">
+<contactref element="U$6" pad="3"/>
+<contactref element="COOLANT.JP" pad="4"/>
+<wire x1="-173.99" y1="-372.42" x2="-167.64" y2="-394.97" width="0" layer="19" extent="1-1"/>
+</signal>
+<signal name="N$13">
+<contactref element="U$5" pad="4"/>
+<contactref element="COOLANT.JP" pad="1"/>
+<wire x1="-167.64" y1="-372.42" x2="-175.26" y2="-394.97" width="0" layer="19" extent="1-1"/>
+</signal>
+<signal name="N$15">
+<contactref element="COOLANT.JP" pad="3"/>
+<contactref element="U$6" pad="4"/>
+<wire x1="-176.53" y1="-372.42" x2="-170.18" y2="-394.97" width="0" layer="19" extent="1-1"/>
+</signal>
+<signal name="N$36">
+<contactref element="LED6" pad="C"/>
+<contactref element="R6" pad="1"/>
+<wire x1="-177.93" y1="-400.05" x2="-182.88" y2="-397.03" width="0" layer="19" extent="1-1"/>
+</signal>
+<signal name="N$37">
+<contactref element="R6" pad="2"/>
+<contactref element="U$6" pad="1"/>
+<wire x1="-176.53" y1="-381.96" x2="-175.13" y2="-400.05" width="0" layer="19" extent="1-1"/>
+</signal>
 </signals>

Commit message: 20180510
Parts:
- removed JP1: (no value), pinhead:2X09/90
- added SENSOR.JP: (no value), pinhead:2X09/90
- moved COOLANT.JP 628.0 mm to (231.1, 90.8)
- moved EXT.JP 628.0 mm to (278.0, 111.2)
- moved LED.X.1 628.0 mm to (283.1, 141.6)
- moved LED.X.2 628.0 mm to (276.8, 135.3)
- moved LED.Y.1 628.0 mm to (295.8, 162.0)
- moved LED.Y.2 628.0 mm to (289.5, 148.0)
- moved LED.Z.1 628.0 mm to (270.4, 128.9)
- moved LED.Z.2 628.0 mm to (264.1, 122.6)
- moved LED1 628.0 mm to (332.6, 245.8)
- moved LED2 628.0 mm to (326.3, 245.8)
- moved LED3 628.0 mm to (319.9, 245.8)
- moved LED4 628.0 mm to (313.6, 245.8)
- moved LED5 628.0 mm to (243.8, 101.0)
- moved LED6 628.0 mm to (219.6, 83.2)
- moved PROBE 628.0 mm to (304.7, 179.7)
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Connections:
- removed net +12V: EXT.JP.1, EXT.JP.2, EXT.JP.7, EXT.JP.8, JP1.1, JP1.13, JP1.14, JP1.2, JP1.7, JP1.8, PWR.JP.1
- removed net GND: EXT.JP.11, EXT.JP.12, EXT.JP.5, EXT.JP.6, JP1.11, JP1.12, JP1.17, JP1.18, JP1.5, JP1.6, PROBE.2, PWR.JP.3, U$1.2, U$1.3, U$2.2, U$2.3, U$3.2, U$3.3, U$4.2, U$4.3, U$5.2, U$6.2, U1.X.2, U1.X.3, U1.Y.2, U1.Y.3, U1.Z.2, U1.Z.3, U2.X.2, U2.X.3, U2.Y.2, U2.Y.3, U2.Z.2, U2.Z.3, X2.P$4
- net MEGA2560.GND: now also EXT.JP.11, EXT.JP.12, EXT.JP.5, EXT.JP.6, PROBE.2, PWR.JP.3, SENSOR.JP.11, SENSOR.JP.12, SENSOR.JP.17, SENSOR.JP.18, SENSOR.JP.5, SENSOR.JP.6, U$1.2, U$1.3, U$2.2, U$2.3, U$3.2, U$3.3, U$4.2, U$4.3, U$5.2, U$6.2, U1.X.2, U1.X.3, U1.Y.2, U1.Y.3, U1.Z.2, U1.Z.3, U2.X.2, U2.X.3, U2.Y.2, U2.Y.3, U2.Z.2, U2.Z.3, X2.P$4
- net MEGA2560.VIN.12V: now also EXT.JP.1, EXT.JP.2, EXT.JP.7, EXT.JP.8, PWR.JP.1, SENSOR.JP.1, SENSOR.JP.13, SENSOR.JP.14, SENSOR.JP.2, SENSOR.JP.7, SENSOR.JP.8
- net SENSOR.LIMIT.X.1: now also SENSOR.JP.3; no longer JP1.3
- net SENSOR.LIMIT.X.2: now also SENSOR.JP.4; no longer JP1.4
- net SENSOR.LIMIT.Y.1: now also SENSOR.JP.9; no longer JP1.9
- net SENSOR.LIMIT.Y.2: now also SENSOR.JP.10; no longer JP1.10
- net SENSOR.LIMIT.Z.1: now also SENSOR.JP.15; no longer JP1.15
- net SENSOR.LIMIT.Z.2: now also SENSOR.JP.16; no longer JP1.16
Routing:
- net MEGA2560.D30.DIR.X: track 0.00 -> 656.7 mm
- net +5V: track 0.00 -> 54.0 mm
- net MEGA2560.D13.STEPPER.EN: track 0.00 -> 53.2 mm
- net MEGA2560.D32.DIR.Z: track 0.00 -> 39.6 mm, vias 0 -> 1
- net MEGA2560.D24.STEP.X: track 0.00 -> 18.4 mm
Other:
- board size 160 x 100 mm -> 402.5 x 482 mm

Commit message: 20180511
Parts:
- removed U$1, U$2, U$3, U$4: LTV817LTV817S, net173:DIL4-SMD
- removed X1: (no value), con-molex-micro-fit-3_0:43045-0800
- added ABORT, HOLD, SAFETY.DOOR, START: LTV817LTV817S, net173:DIL4-SMD
- added JP1: (no value), pinhead:2X04
- EXT.JP: device pinhead:2X11/90 -> pinhead:2X11
- SENSOR.JP: device pinhead:2X09/90 -> pinhead:2X09
- moved U1.X 499.8 mm to (132.1, 64.8)
- moved U2.X 492.6 mm to (137.2, 64.8)
- moved U2.Y 410.4 mm to (127.0, 64.8)
- moved U1.Y 408.1 mm to (121.9, 64.8)
- moved U2.Z 392.2 mm to (116.8, 64.8)
- moved U1.Z 389.6 mm to (111.8, 64.8)
- moved R2 329.6 mm to (128.3, 6.35), turned to 180 degrees
- moved R3 321.8 mm to (128.3, 11.4), turned to 180 degrees
- moved LED1 311.4 mm to (121.9, 16.5), turned to 90 degrees
- moved R4 310.5 mm to (128.3, 21.6), turned to 180 degrees
- moved R5 310.5 mm to (128.3, 16.5), turned to 180 degrees
- moved LED3 306.8 mm to (121.9, 11.4), turned to 90 degrees
- moved LED4 306.7 mm to (121.9, 6.35), turned to 90 degrees
- moved LED2 303.4 mm to (121.9, 21.6), turned to 90 degrees
- moved PROBE 254.8 mm to (166.4, -34.3), turned to 270 degrees
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- renumbered U$5 to FLOOD, U$6 to MIST
Connections:
- net +5V: now also JP1.2, JP1.4, JP1.6, JP1.8; no longer X1.P$1, X1.P$2, X1.P$3, X1.P$4
- net MEGA2560.A10.CYCLE.START: now also START.4; no longer U$3.4
- net MEGA2560.A11.SAFETY.DOOR: now also SAFETY.DOOR.4; no longer U$4.4
- net MEGA2560.A8.RESET.ABORT: now also ABORT.4; no longer U$1.4
- net MEGA2560.A9.FEED.HOLD: now also HOLD.4; no longer U$2.4
- net MEGA2560.D8.COOLANT.FLOOD: now also R1.1; no longer LED5.A
- net MEGA2560.D9.COOLANT.MIST: now also R6.1; no longer LED6.A
- net MEGA2560.GND: now also ABORT.2, ABORT.3, HOLD.2, HOLD.3, SAFETY.DOOR.2, SAFETY.DOOR.3, START.2, START.3; no longer U$1.2, U$1.3, U$2.2, U$2.3, U$3.2, U$3.3, U$4.2, U$4.3
- net N$19: now also ABORT.1, LED2.C; no longer LED2.A, X1.P$8
- net N$2: now also LED5.A; no longer FLOOD.1
- net N$20: now also JP1.3, R5.1; no longer LED1.A, X1.P$7
- net N$21: now also JP1.5, R3.1; no longer LED3.A, X1.P$6
- net N$22: now also HOLD.1, LED1.C; no longer LED2.C, R4.1
- net N$23: now also LED1.A, R5.2; no longer R4.2, U$1.1
- net N$24: now also LED2.A, R4.2; no longer R5.2, U$2.1
- net N$30: now also JP1.1, R4.1; no longer LED1.C, R5.1
- net N$31: now also JP1.7, R2.1; no longer LED4.A, X1.P$5
- net N$32: now also LED3.A, R3.2; no longer LED3.C, R3.1
- net N$33: now also LED3.C, START.1; no longer LED4.C, R2.1
- net N$34: now also LED4.C, SAFETY.DOOR.1; no longer R2.2, U$4.1
- net N$35: now also LED4.A, R2.2; no longer R3.2, U$3.1
- net N$36: now also LED6.A, R6.2; no longer LED6.C, R6.1
- net N$37: now also LED6.C; no longer MIST.1, R6.2
- net N$4: now also FLOOD.1; no longer R1.1
Routing:
- net MEGA2560.D30.DIR.X: track 656.7 -> 56.2 mm
- net MEGA2560.GND: track 0.00 -> 251.7 mm, vias 0 -> 4
- net MEGA2560.VIN.12V: track 0.00 -> 132.4 mm, vias 0 -> 2
- net MEGA2560.D1.TXD0: track 0.00 -> 71.4 mm, vias 0 -> 1
- net MEGA2560.D0.RXD0: track 0.00 -> 64.6 mm, vias 0 -> 1
- net MEGA2560.D12.LIMIT.Z: track 0.00 -> 57.1 mm
- net MEGA2560.D11.LIMIT.Y: track 0.00 -> 47.7 mm
- net MEGA2560.D10.LIMIT.X: track 0.00 -> 37.5 mm
- net +5V: track 54.0 -> 77.9 mm
- net MEGA2560.D31.DIR.Y: track 0.00 -> 16.1 mm
- net N$30: track 0.00 -> 15.6 mm, vias 0 -> 1
- net MEGA2560.D26.STEP.Z: track 0.00 -> 15.5 mm
- net MEGA2560.D32.DIR.Z: track 39.6 -> 24.7 mm, vias 1 -> 0
- net MEGA2560.D24.STEP.X: track 18.4 -> 32.2 mm
- net MEGA2560.A11.SAFETY.DOOR: track 0.00 -> 13.3 mm
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Other:
- board size 402.5 x 482 mm -> 160 x 106.3 mm

Commit message: 20180511
Parts:
- moved R6 25.6 mm to (236.2, 105.4), turned to 180 degrees
- moved LED6 24.4 mm to (229.9, 105.4), turned to 90 degrees
- moved R1 18.6 mm to (236.2, 110.5), turned to 180 degrees
- moved LED5 16.8 mm to (229.9, 110.5), turned to 90 degrees
- moved FLOOD 16.7 mm to (221.0, 111.8), turned to 90 degrees
- moved MIST 6.53 mm to (221.0, 106.7), turned to 90 degrees
Connections:
- net N$37: now also MIST.1
Routing:
- net MEGA2560.GND: track 251.7 -> 370.8 mm, vias 4 -> 5
- net MEGA2560.D10.LIMIT.X: track 37.5 -> 105.2 mm, vias 0 -> 1
- net MEGA2560.D11.LIMIT.Y: track 47.7 -> 102.6 mm, vias 0 -> 1
- net MEGA2560.D12.LIMIT.Z: track 57.1 -> 66.0 mm, vias 0 -> 1
- net N$36: track 0.00 -> 3.20 mm
- net N$2: track 0.00 -> 3.20 mm
- net N$4: track 0.00 -> 2.37 mm
- net N$37: track 0.00 -> 2.37 mm

Commit message: 20180511
Parts:
- moved R1 100.4 mm to (153.7, 53.3), turned to 0 degrees
- moved COOLANT.JP 98.5 mm to (166.4, 75.6)
- moved R6 96.3 mm to (153.7, 55.9), turned to 0 degrees
- moved LED5 91.2 mm to (158.8, 53.3), turned to 270 degrees
- moved LED6 87.8 mm to (154.9, 59.7), turned to 0 degrees
- moved FLOOD 78.4 mm to (161.3, 61.0), turned to 0 degrees
- moved MIST 75.1 mm to (156.2, 68.6), turned to 0 degrees
- moved STEPPER-X1 28.3 mm to (173.8, 31.0)
- moved STEPPER-X2 28.3 mm to (173.8, 15.0)
- moved STEPPER-Y 28.3 mm to (173.8, -1.00)
- moved STEPPER-Z 28.3 mm to (173.8, -17.0)
- moved X2 26.5 mm to (168.7, 47.0)
- moved PWR.JP 7.07 mm to (167.4, 90.8)
- moved EXT.JP 2.54 mm to (124.5, 82.5)
Connections:
- net N$13: now also COOLANT.JP.2; no longer COOLANT.JP.1
- net N$15: now also COOLANT.JP.4; no longer COOLANT.JP.3
- net N$6: now also COOLANT.JP.1; no longer COOLANT.JP.2
- net N$9: now also COOLANT.JP.3; no longer COOLANT.JP.4
Routing:
- net MEGA2560.GND: track 370.8 -> 418.0 mm, vias 5 -> 6
- net MEGA2560.D6.SPINDLE.EN: track 0.00 -> 24.5 mm, vias 0 -> 1
- net N$6: track 0.00 -> 20.4 mm
- net MEGA2560.D7.SPINDLE.PWM: track 0.00 -> 18.3 mm, vias 0 -> 1
- net N$13: track 0.00 -> 16.8 mm
- net N$15: track 0.00 -> 11.2 mm
- net MEGA2560.D5.SPINDLE.DIR: track 0.00 -> 6.35 mm
- net N$9: track 0.00 -> 5.55 mm
- net MEGA2560.VIN.12V: track 132.4 -> 129.8 mm
- net MEGA2560.D11.LIMIT.Y: track 102.6 -> 100.1 mm
- net MEGA2560.D10.LIMIT.X: track 105.2 -> 102.6 mm
- net MEGA2560.D1.TXD0: track 71.4 -> 68.9 mm
- net MEGA2560.D12.LIMIT.Z: track 66.0 -> 63.5 mm
- net MEGA2560.D0.RXD0: track 64.6 -> 62.0 mm
- net N$2: track 3.20 -> 1.93 mm
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Other:
- board size 160 x 106.3 mm -> 164 x 128 mm

Commit message: 20180513
Parts:
- PROBE: device pinhead:1X02/90 -> pinhead:1X02
- moved PROBE 62.0 mm to (109.2, -10.2), turned to 180 degrees
- moved STEPPER-X1 5.10 mm to (168.8, 32.0)
- moved STEPPER-X2 5.10 mm to (168.8, 16.0)
- moved STEPPER-Y 5.10 mm to (168.8, 0.00)
- moved STEPPER-Z 5.10 mm to (168.8, -16.0)
- moved PWR.JP 0.94 mm to (166.4, 90.8)
- moved X2 0.08 mm to (168.8, 47.0)
Connections:
- new net GND: ABORT.2, HOLD.2, PROBE.1, SAFETY.DOOR.2, START.2
- new net MEGA2560.GND.INT.1: JP.MEGA2560.PWM.HIGH.4
- net MEGA2560.A15.PROBE: now also PROBE.2; no longer PROBE.1
- net MEGA2560.GND: no longer ABORT.2, HOLD.2, JP.MEGA2560.PWM.HIGH.4, PROBE.2, SAFETY.DOOR.2, START.2
Routing:
- net +5V: track 77.9 -> 270.3 mm, vias 0 -> 4
- net MEGA2560.VIN.12V: track 129.8 -> 201.1 mm, vias 2 -> 5
- net MEGA2560.GND: track 418.0 -> 484.6 mm, vias 6 -> 7
- net MEGA2560.D13.STEPPER.EN: track 53.2 -> 113.1 mm, vias 0 -> 3
- net GND: track 0.00 -> 59.5 mm, vias 0 -> 1
- net MEGA2560.D24.STEP.X: track 32.2 -> 72.5 mm, vias 0 -> 1
- net MEGA2560.D30.DIR.X: track 56.2 -> 92.9 mm, vias 0 -> 1
- net MEGA2560.A15.PROBE: track 0.00 -> 20.5 mm, vias 0 -> 1
- net MEGA2560.D31.DIR.Y: track 16.1 -> 36.2 mm, vias 0 -> 1
- net MEGA2560.D26.STEP.Z: track 15.5 -> 35.3 mm, vias 0 -> 1
- net MEGA2560.D32.DIR.Z: track 24.7 -> 43.1 mm, vias 0 -> 1
- net MEGA2560.D25.STEP.Y: track 9.42 -> 25.2 mm, vias 0 -> 1
- net MEGA2560.D5.SPINDLE.DIR: track 6.35 -> 14.6 mm, vias 0 -> 1
Other:
- board size 164 x 128 mm -> 74.9 x 120.7 mm

Commit message: Auto stash before merge of "master" and "origin/master"
Parts:
- removed J1: AVR_SPI_PROG_3X2PTH, SparkFun-Connectors:2X3
Other:
- outline, holes or cut-outs redrawn
Changed lines of the file:
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@@
 <wire x1="97.79" y1="97.79" x2="97.79" y2="-22.86" width="0" layer="20"/>
 <hole x="127" y="0" drill="0.6"/>
-<wire x1="151.13" y1="-1.27" x2="148.59" y2="-3.81" width="0.254" layer="20"/>
-<wire x1="138.43" y1="-3.81" x2="135.89" y2="-6.35" width="0.254" layer="20"/>
-<wire x1="135.89" y1="-6.35" x2="101.6" y2="-6.35" width="0.254" layer="20"/>
-<wire x1="101.6" y1="-6.35" x2="99.06" y2="-3.81" width="0.254" layer="20"/>
-<wire x1="99.06" y1="-3.81" x2="98.79" y2="-3.81" width="0.254" layer="20"/>
-<wire x1="98.79" y1="-3.81" x2="97.79" y2="-2.81" width="0.254" layer="20" curve="-90"/>
-<wire x1="97.79" y1="-2.81" x2="97.79" y2="94.25" width="0.254" layer="20"/>
-<wire x1="97.79" y1="94.25" x2="98.79" y2="95.25" width="0.254" layer="20" curve="-90"/>
-<wire x1="98.79" y1="95.25" x2="150.13" y2="95.25" width="0.254" layer="20"/>
-<wire x1="150.13" y1="95.25" x2="151.13" y2="94.25" width="0.254" layer="20" curve="-90"/>
-<wire x1="151.13" y1="94.25" x2="151.13" y2="-1.27" width="0.254" layer="20"/>
-<wire x1="148.59" y1="-3.81" x2="138.43" y2="-3.81" width="0.254" layer="20"/>
+<wire x1="151.13" y1="-1.27" x2="148.59" y2="-3.81" width="0.254" layer="48"/>
+<wire x1="138.43" y1="-3.81" x2="135.89" y2="-6.35" width="0.254" layer="48"/>
+<wire x1="135.89" y1="-6.35" x2="101.6" y2="-6.35" width="0.254" layer="48"/>
+<wire x1="101.6" y1="-6.35" x2="99.06" y2="-3.81" width="0.254" layer="48"/>
+<wire x1="99.06" y1="-3.81" x2="98.79" y2="-3.81" width="0.254" layer="48"/>
+<wire x1="98.79" y1="-3.81" x2="97.79" y2="-2.81" width="0.254" layer="48" curve="-90"/>
+<wire x1="97.79" y1="-2.81" x2="97.79" y2="94.25" width="0.254" layer="48"/>
+<wire x1="97.79" y1="94.25" x2="98.79" y2="95.25" width="0.254" layer="48" curve="-90"/>
+<wire x1="98.79" y1="95.25" x2="150.13" y2="95.25" width="0.254" layer="48"/>
+<wire x1="150.13" y1="95.25" x2="151.13" y2="94.25" width="0.254" layer="48" curve="-90"/>
+<wire x1="151.13" y1="94.25" x2="151.13" y2="-1.27" width="0.254" layer="48"/>
+<wire x1="148.59" y1="-3.81" x2="138.43" y2="-3.81" width="0.254" layer="48"/>
 <hole x="100.33" y="-1.27" drill="3.5"/>
 <hole x="148.59" y="5.08" drill="3.5"/>
@@
 <element name="JP.MEGA2560.COMMUNICATION" library="pinhead" package="1X08" value="" x="148.59" y="17.78" rot="R270"/>
 <element name="JP.MEGA2560.PWM.LOW" library="pinhead" package="1X08" value="" x="148.59" y="40.64" rot="R270"/>
-<element name="J1" library="SparkFun-Connectors" package="2X3" value="AVR_SPI_PROG_3X2PTH" x="128.27" y="31.75" rot="R180"/>
 <element name="U1.X" library="net173" package="DIL4-SMD" value="LTV817LTV817S" x="132.08" y="64.77"/>
 <element name="U2.X" library="net173" package="DIL4-SMD" value="LTV817LTV817S" x="137.16" y="64.77"/>
