File: EAGLE/!PRJ/Control.Board/Control.Board.sch (EAGLE design)
At the start: 50 parts, among them J1 AVR_SPI_PROG_3X2PTH, U1.X LTV817LTV817S, U1.Y LTV817LTV817S, U1.Z LTV817LTV817S, U2.X LTV817LTV817S, U2.Y LTV817LTV817S, U2.Z LTV817LTV817S

Commit message: 20180505
Parts:
- removed JP.LIMIT.X, JP.LIMIT.Y, JP.LIMIT.Z: (no value), pinhead:PINHD-1X6
- removed LED1.X, LED1.Y, LED1.Z, LED2.X, LED2.Y, LED2.Z: (no value), led:LEDCHIPLED_0805
- removed R1: (no value), rcl:R-EU_M1206
- removed R1.X, R1.Y, R1.Z, R2.X, R2.Y, R2.Z: 470, rcl:R-EU_M0805
- removed R3.X, R3.Y, R3.Z: 10K, rcl:R-EU_M0805
- added EXT.JP: (no value), pinhead:PINHD-2X11/90
- added JP1: (no value), pinhead:PINHD-2X9/90
- added LED.X.1, LED.X.2, LED.Y.1, LED.Y.2, LED.Z.1, LED.Z.2: (no value), led:LEDCHIPLED_1206
- added PROBE: (no value), pinhead:PINHD-1X2/90
- added PWR.JP: (no value), pinhead:PINHD-1X3/90
- added R.X.1, R.X.2, R.Y.1, R.Y.2, R.Z.1, R.Z.2: 470, rcl:R-EU_M1206
Connections:
- removed net N$13: JP.LIMIT.Z.2, R1.Z.1
- removed net N$15: JP.LIMIT.Z.5, R2.Z.1
- removed net N$2: JP.LIMIT.Y.2, R1.Y.1
- removed net N$4: JP.LIMIT.X.2, R1.X.1
- removed net N$6: JP.LIMIT.X.5, R2.X.1
- removed net N$9: JP.LIMIT.Y.5, R2.Y.1
- new net SENSOR.LIMIT.X.1: JP1.3, R.X.1.1
- new net SENSOR.LIMIT.X.2: JP1.4, R.X.2.1
- new net SENSOR.LIMIT.Y.1: JP1.9, R.Y.1.1
- new net SENSOR.LIMIT.Y.2: JP1.10, R.Y.2.1
- new net SENSOR.LIMIT.Z.1: JP1.15, R.Z.1.1
- new net SENSOR.LIMIT.Z.2: JP1.16, R.Z.2.1
- net +12V: now also EXT.JP.1, EXT.JP.2, EXT.JP.7, EXT.JP.8, JP1.1, JP1.13, JP1.14, JP1.2, JP1.7, JP1.8, PWR.JP.1; no longer JP.LIMIT.X.1, JP.LIMIT.X.4, JP.LIMIT.Y.1, JP.LIMIT.Y.4, JP.LIMIT.Z.1, JP.LIMIT.Z.4
- net +5V: now also EXT.JP.10, EXT.JP.3, EXT.JP.4, EXT.JP.9, PWR.JP.2; no longer R3.X.2, R3.Y.2, R3.Z.2
- net GND: now also EXT.JP.11, EXT.JP.12, EXT.JP.5, EXT.JP.6, JP1.11, JP1.12, JP1.17, JP1.18, JP1.5, JP1.6, PROBE.2, PWR.JP.3; no longer JP.LIMIT.X.3, JP.LIMIT.X.6, JP.LIMIT.Y.3, JP.LIMIT.Y.6, JP.LIMIT.Z.3, JP.LIMIT.Z.6
- net MEGA2560.A15.PROBE: now also PROBE.1
- net MEGA2560.D0.RXD0: now also EXT.JP.21, EXT.JP.22
- net MEGA2560.D1.TXD0: now also EXT.JP.19, EXT.JP.20
- net MEGA2560.D10.LIMIT.X: now also EXT.JP.13, EXT.JP.14; no longer R3.X.1
- net MEGA2560.D11.LIMIT.Y: now also EXT.JP.15, EXT.JP.16; no longer R3.Y.1
- net MEGA2560.D12.LIMIT.Z: now also EXT.JP.17, EXT.JP.18; no longer R3.Z.1
- net N$1: now also LED.X.2.C; no longer LED2.X.C
- net N$10: now also LED.Y.2.A, R.Y.2.2; no longer LED2.Y.A, R2.Y.2
- net N$11: now also LED.Y.2.C; no longer LED2.Y.C
- net N$12: now also LED.Y.1.C; no longer LED1.Y.C
- net N$14: now also LED.Z.1.A, R.Z.1.2; no longer LED1.Z.A, R1.Z.2
- net N$16: now also LED.Z.2.A, R.Z.2.2; no longer LED2.Z.A, R2.Z.2
- net N$17: now also LED.Z.2.C; no longer LED2.Z.C
- net N$18: now also LED.Z.1.C; no longer LED1.Z.C
- net N$3: now also LED.Y.1.A, R.Y.1.2; no longer LED1.Y.A, R1.Y.2
- net N$5: now also LED.X.1.A, R.X.1.2; no longer LED1.X.A, R1.X.2
- net N$7: now also LED.X.2.A, R.X.2.2; no longer LED2.X.A, R2.X.2
- net N$8: now also LED.X.1.C; no longer LED1.X.C

Commit message: 20180510
Parts:
- added COOLANT.JP: (no value), pinhead:PINHD-1X4/90
- added LED5, LED6: (no value), led:LEDCHIPLED_1206
- added R1, R6: 100, rcl:R-EU_M1206
- added U$5, U$6: LTV817LTV817S, net173:LTV817LTV817S
- added X2: (no value), con-molex-micro-fit-3_0:HEADER_POS4_43045-0401
Connections:
- new net N$13: COOLANT.JP.1, U$5.COL
- new net N$15: COOLANT.JP.3, U$6.COL
- new net N$2: R1.2, U$5.A
- new net N$36: LED6.C, R6.1
- new net N$37: R6.2, U$6.A
- new net N$4: LED5.C, R1.1
- new net N$6: COOLANT.JP.2, U$5.EMIT
- new net N$9: COOLANT.JP.4, U$6.EMIT
- net GND: now also U$5.C, U$6.C, X2.4
- net MEGA2560.D5.SPINDLE.DIR: now also X2.3
- net MEGA2560.D6.SPINDLE.EN: now also X2.2
- net MEGA2560.D7.SPINDLE.PWM: now also X2.1
- net MEGA2560.D8.COOLANT.FLOOD: now also LED5.A
- net MEGA2560.D9.COOLANT.MIST: now also LED6.A
Changed lines of the file:
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@@
 <setting verticaltext="up"/>
 </settings>
-<grid distance="0.1" unitdist="inch" unit="inch" style="lines" multiple="1" display="yes" altdistance="0.01" altunitdist="inch" altunit="inch"/>
+<grid distance="0.1" unitdist="inch" unit="inch" style="lines" multiple="1" display="no" altdistance="0.01" altunitdist="inch" altunit="inch"/>
 <layers>
 <layer number="1" name="Top" color="4" fill="1" visible="no" active="no"/>
@@
 <part name="P+5" library="supply1" deviceset="+12V" device=""/>
 <part name="P+6" library="supply1" deviceset="+5V" device=""/>
+<part name="R1" library="rcl" deviceset="R-EU_" device="M1206" value="100"/>
+<part name="LED5" library="led" deviceset="LED" device="CHIPLED_1206"/>
+<part name="U$5" library="net173" deviceset="LTV817" device="LTV817S"/>
+<part name="U$6" library="net173" deviceset="LTV817" device="LTV817S"/>
+<part name="GND21" library="supply1" deviceset="GND" device=""/>
+<part name="COOLANT.JP" library="pinhead" deviceset="PINHD-1X4" device="/90"/>
+<part name="R6" library="rcl" deviceset="R-EU_" device="M1206" value="100"/>
+<part name="LED6" library="led" deviceset="LED" device="CHIPLED_1206"/>
+<part name="X2" library="con-molex-micro-fit-3_0" deviceset="HEADER_POS4_?" device="43045-0401"/>
+<part name="GND11" library="supply1" deviceset="GND" device=""/>
 </parts>
 <sheets>
@@
 </segment>
 </net>
+</nets>
+</sheet>
+<sheet>
+<description>Coolant</description>
+<plain>
+</plain>
+<instances>
+<instance part="R1" gate="G$1" x="53.34" y="73.66"/>
+<instance part="LED5" gate="G$1" x="35.56" y="73.66" rot="R90"/>
+<instance part="U$5" gate="G$1" x="78.74" y="71.12"/>
+<instance part="U$6" gate="G$1" x="78.74" y="43.18"/>
+<instance part="GND21" gate="1" x="63.5" y="33.02"/>
+<instance part="COOLANT.JP" gate="A" x="111.76" y="68.58"/>
+<instance part="R6" gate="G$1" x="53.34" y="45.72"/>
+<instance part="LED6" gate="G$1" x="35.56" y="45.72" rot="R90"/>
+</instances>
+<busses>
+</busses>
+<nets>
+<net name="N$2" class="0">
+<segment>
+<pinref part="U$5" gate="G$1" pin="A"/>
+<pinref part="R1" gate="G$1" pin="2"/>
+<wire x1="68.58" y1="73.66" x2="58.42" y2="73.66" width="0.1524" layer="91"/>
+</segment>
+</net>
+<net name="N$4" class="0">
+<segment>
+<pinref part="R1" gate="G$1" pin="1"/>
+<pinref part="LED5" gate="G$1" pin="C"/>
+<wire x1="48.26" y1="73.66" x2="40.64" y2="73.66" width="0.1524" layer="91"/>
+</segment>
+</net>
+<net name="N$6" class="0">
+<segment>
+<pinref part="U$5" gate="G$1" pin="EMIT"/>
+<wire x1="86.36" y1="68.58" x2="91.44" y2="68.58" width="0.1524" layer="91"/>
+<wire x1="91.44" y1="68.58" x2="91.44" y2="71.12" width="0.1524" layer="91"/>
+<pinref part="COOLANT.JP" gate="A" pin="2"/>
+<wire x1="91.44" y1="71.12" x2="109.22" y2="71.12" width="0.1524" layer="91"/>
+</segment>
+</net>
+<net name="N$9" class="0">
+<segment>
+<pinref part="U$6" gate="G$1" pin="EMIT"/>
+<wire x1="86.36" y1="40.64" x2="96.52" y2="40.64" width="0.1524" layer="91"/>
+<wire x1="96.52" y1="40.64" x2="96.52" y2="66.04" width="0.1524" layer="91"/>
+<pinref part="COOLANT.JP" gate="A" pin="4"/>
+<wire x1="96.52" y1="66.04" x2="109.22" y2="66.04" width="0.1524" layer="91"/>
+</segment>
+</net>
+<net name="GND" class="0">
+<segment>
+<pinref part="U$5" gate="G$1" pin="C"/>
+<pinref part="GND21" gate="1" pin="GND"/>
+<wire x1="68.58" y1="68.58" x2="63.5" y2="68.58" width="0.1524" layer="91"/>
+<wire x1="63.5" y1="68.58" x2="63.5" y2="40.64" width="0.1524" layer="91"/>
+<pinref part="U$6" gate="G$1" pin="C"/>
+<wire x1="63.5" y1="40.64" x2="63.5" y2="35.56" width="0.1524" layer="91"/>
+<wire x1="68.58" y1="40.64" x2="63.5" y2="40.64" width="0.1524" layer="91"/>
+<junction x="63.5" y="40.64"/>
+</segment>
+</net>
+<net name="N$13" class="0">
+<segment>
+<pinref part="U$5" gate="G$1" pin="COL"/>
+<pinref part="COOLANT.JP" gate="A" pin="1"/>
+<wire x1="86.36" y1="73.66" x2="109.22" y2="73.66" width="0.1524" layer="91"/>
+</segment>
+</net>
+<net name="N$15" class="0">
+<segment>
+<pinref part="COOLANT.JP" gate="A" pin="3"/>
+<wire x1="109.22" y1="68.58" x2="93.98" y2="68.58" width="0.1524" layer="91"/>
+<wire x1="93.98" y1="68.58" x2="93.98" y2="45.72" width="0.1524" layer="91"/>
+<pinref part="U$6" gate="G$1" pin="COL"/>
+<wire x1="93.98" y1="45.72" x2="86.36" y2="45.72" width="0.1524" layer="91"/>
+</segment>
+</net>
+<net name="N$36" class="0">
+<segment>
+<pinref part="LED6" gate="G$1" pin="C"/>
+<pinref part="R6" gate="G$1" pin="1"/>
+<wire x1="40.64" y1="45.72" x2="48.26" y2="45.72" width="0.1524" layer="91"/>
+</segment>
+</net>
+<net name="N$37" class="0">
+<segment>
+<pinref part="R6" gate="G$1" pin="2"/>
+<pinref part="U$6" gate="G$1" pin="A"/>
+<wire x1="58.42" y1="45.72" x2="68.58" y2="45.72" width="0.1524" layer="91"/>
+</segment>
+</net>
+<net name="MEGA2560.D8.COOLANT.FLOOD" class="0">
+<segment>
+<pinref part="LED5" gate="G$1" pin="A"/>
+<wire x1="33.02" y1="73.66" x2="25.4" y2="73.66" width="0.1524" layer="91"/>
+<label x="25.4" y="73.66" size="0.8128" layer="95" rot="R180" xref="yes"/>
+</segment>
+</net>
+<net name="MEGA2560.D9.COOLANT.MIST" class="0">
+<segment>
+<pinref part="LED6" gate="G$1" pin="A"/>
+<wire x1="33.02" y1="45.72" x2="25.4" y2="45.72" width="0.1524" layer="91"/>
+<label x="25.4" y="45.72" size="0.8128" layer="95" rot="R180" xref="yes"/>
+</segment>
+</net>
+</nets>
+</sheet>
+<sheet>
+<description>Spindle</description>
+<plain>
+</plain>
+<instances>
+<instance part="X2" gate="G$1" x="86.36" y="71.12"/>
+<instance part="GND11" gate="1" x="76.2" y="60.96"/>
+</instances>
+<busses>
+</busses>
+<nets>
+<net name="MEGA2560.D7.SPINDLE.PWM" class="0">
+<segment>
+<pinref part="X2" gate="G$1" pin="1"/>
+<wire x1="81.28" y1="76.2" x2="48.26" y2="76.2" width="0.1524" layer="91"/>
+<label x="48.26" y="76.2" size="0.8128" layer="95" rot="R180" xref="yes"/>
+</segment>
+</net>
+<net name="MEGA2560.D6.SPINDLE.EN" class="0">
+<segment>
+<pinref part="X2" gate="G$1" pin="2"/>
+<wire x1="81.28" y1="73.66" x2="48.26" y2="73.66" width="0.1524" layer="91"/>
+<label x="48.26" y="73.66" size="0.8128" layer="95" rot="R180" xref="yes"/>
+</segment>
+</net>
+<net name="MEGA2560.D5.SPINDLE.DIR" class="0">
+<segment>
+<pinref part="X2" gate="G$1" pin="3"/>
+<wire x1="81.28" y1="71.12" x2="48.26" y2="71.12" width="0.1524" layer="91"/>
+<label x="48.26" y="71.12" size="0.8128" layer="95" rot="R180" xref="yes"/>
+</segment>
+</net>
+<net name="GND" class="0">
+<segment>
+<pinref part="X2" gate="G$1" pin="4"/>
+<pinref part="GND11" gate="1" pin="GND"/>
+<wire x1="81.28" y1="68.58" x2="76.2" y2="68.58" width="0.1524" layer="91"/>
+<wire x1="76.2" y1="68.58" x2="76.2" y2="63.5" width="0.1524" layer="91"/>
+</segment>
+</net>

Commit message: 20180510
Parts:
- renumbered JP1 to SENSOR.JP
Connections:
- removed net +12V: EXT.JP.1, EXT.JP.2, EXT.JP.7, EXT.JP.8, PWR.JP.1, SENSOR.JP.1, SENSOR.JP.13, SENSOR.JP.14, SENSOR.JP.2, SENSOR.JP.7, SENSOR.JP.8
- removed net GND: EXT.JP.11, EXT.JP.12, EXT.JP.5, EXT.JP.6, PROBE.2, PWR.JP.3, SENSOR.JP.11, SENSOR.JP.12, SENSOR.JP.17, SENSOR.JP.18, SENSOR.JP.5, SENSOR.JP.6, U$1.C, U$1.EMIT, U$2.C, U$2.EMIT, U$3.C, U$3.EMIT, U$4.C, U$4.EMIT, U$5.C, U$6.C, U1.X.C, U1.X.EMIT, U1.Y.C, U1.Y.EMIT, U1.Z.C, U1.Z.EMIT, U2.X.C, U2.X.EMIT, U2.Y.C, U2.Y.EMIT, U2.Z.C, U2.Z.EMIT, X2.4
- net MEGA2560.GND: now also EXT.JP.11, EXT.JP.12, EXT.JP.5, EXT.JP.6, PROBE.2, PWR.JP.3, SENSOR.JP.11, SENSOR.JP.12, SENSOR.JP.17, SENSOR.JP.18, SENSOR.JP.5, SENSOR.JP.6, U$1.C, U$1.EMIT, U$2.C, U$2.EMIT, U$3.C, U$3.EMIT, U$4.C, U$4.EMIT, U$5.C, U$6.C, U1.X.C, U1.X.EMIT, U1.Y.C, U1.Y.EMIT, U1.Z.C, U1.Z.EMIT, U2.X.C, U2.X.EMIT, U2.Y.C, U2.Y.EMIT, U2.Z.C, U2.Z.EMIT, X2.4
- net MEGA2560.VIN.12V: now also EXT.JP.1, EXT.JP.2, EXT.JP.7, EXT.JP.8, PWR.JP.1, SENSOR.JP.1, SENSOR.JP.13, SENSOR.JP.14, SENSOR.JP.2, SENSOR.JP.7, SENSOR.JP.8
Changed lines of the file:
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@@
 <part name="PROBE" library="pinhead" deviceset="PINHD-1X2" device="/90"/>
 <part name="GND17" library="supply1" deviceset="GND" device=""/>
-<part name="JP1" library="pinhead" deviceset="PINHD-2X9" device="/90"/>
+<part name="SENSOR.JP" library="pinhead" deviceset="PINHD-2X9" device="/90"/>
 <part name="P+3" library="supply1" deviceset="+12V" device=""/>
 <part name="GND18" library="supply1" deviceset="GND" device=""/>
@@
 <part name="X2" library="con-molex-micro-fit-3_0" deviceset="HEADER_POS4_?" device="43045-0401"/>
 <part name="GND11" library="supply1" deviceset="GND" device=""/>
+<part name="GND22" library="supply1" deviceset="GND" device=""/>
+<part name="P+9" library="supply1" deviceset="+12V" device=""/>
 </parts>
 <sheets>
@@
 <instance part="U2.Z" gate="G$1" x="-2.54" y="-35.56"/>
 <instance part="FRAME1" gate="G$1" x="-101.6" y="-78.74"/>
-<instance part="JP1" gate="A" x="88.9" y="-15.24"/>
+<instance part="SENSOR.JP" gate="A" x="88.9" y="-15.24"/>
 <instance part="P+3" gate="1" x="73.66" y="5.08"/>
 <instance part="GND18" gate="1" x="76.2" y="-35.56"/>
@@
 </busses>
 <nets>
-<net name="GND" class="0">
+<net name="MEGA2560.GND" class="0">
 <segment>
 <pinref part="GND4" gate="1" pin="GND"/>
@@
 <pinref part="GND18" gate="1" pin="GND"/>
 <wire x1="76.2" y1="-33.02" x2="76.2" y2="-25.4" width="0.1524" layer="91"/>
-<pinref part="JP1" gate="A" pin="17"/>
+<pinref part="SENSOR.JP" gate="A" pin="17"/>
 <wire x1="76.2" y1="-25.4" x2="86.36" y2="-25.4" width="0.1524" layer="91"/>
 <wire x1="76.2" y1="-25.4" x2="76.2" y2="-17.78" width="0.1524" layer="91"/>
-<pinref part="JP1" gate="A" pin="11"/>
+<pinref part="SENSOR.JP" gate="A" pin="11"/>
 <wire x1="76.2" y1="-17.78" x2="86.36" y2="-17.78" width="0.1524" layer="91"/>
-<pinref part="JP1" gate="A" pin="5"/>
+<pinref part="SENSOR.JP" gate="A" pin="5"/>
 <wire x1="86.36" y1="-10.16" x2="76.2" y2="-10.16" width="0.1524" layer="91"/>
 <wire x1="76.2" y1="-10.16" x2="76.2" y2="-17.78" width="0.1524" layer="91"/>
@@
 </segment>
 <segment>
-<pinref part="JP1" gate="A" pin="6"/>
+<pinref part="SENSOR.JP" gate="A" pin="6"/>
 <pinref part="GND20" gate="1" pin="GND"/>
 <wire x1="93.98" y1="-10.16" x2="104.14" y2="-10.16" width="0.1524" layer="91"/>
 <wire x1="104.14" y1="-10.16" x2="104.14" y2="-17.78" width="0.1524" layer="91"/>
-<pinref part="JP1" gate="A" pin="12"/>
+<pinref part="SENSOR.JP" gate="A" pin="12"/>
 <wire x1="104.14" y1="-17.78" x2="104.14" y2="-25.4" width="0.1524" layer="91"/>
 <wire x1="104.14" y1="-25.4" x2="104.14" y2="-33.02" width="0.1524" layer="91"/>
 <wire x1="93.98" y1="-17.78" x2="104.14" y2="-17.78" width="0.1524" layer="91"/>
-<pinref part="JP1" gate="A" pin="18"/>
+<pinref part="SENSOR.JP" gate="A" pin="18"/>
 <wire x1="93.98" y1="-25.4" x2="104.14" y2="-25.4" width="0.1524" layer="91"/>
 <junction x="104.14" y="-25.4"/>
@@
 </segment>
 </net>
-<net name="+12V" class="0">
-<segment>
-<pinref part="JP1" gate="A" pin="1"/>
+<net name="MEGA2560.VIN.12V" class="0">
+<segment>
+<pinref part="SENSOR.JP" gate="A" pin="1"/>
 <pinref part="P+3" gate="1" pin="+12V"/>
 <wire x1="86.36" y1="-5.08" x2="73.66" y2="-5.08" width="0.1524" layer="91"/>
 <wire x1="73.66" y1="-5.08" x2="73.66" y2="2.54" width="0.1524" layer="91"/>
-<pinref part="JP1" gate="A" pin="7"/>
+<pinref part="SENSOR.JP" gate="A" pin="7"/>
 <wire x1="86.36" y1="-12.7" x2="73.66" y2="-12.7" width="0.1524" layer="91"/>
 <wire x1="73.66" y1="-12.7" x2="73.66" y2="-5.08" width="0.1524" layer="91"/>
-<pinref part="JP1" gate="A" pin="13"/>
+<pinref part="SENSOR.JP" gate="A" pin="13"/>
 <wire x1="86.36" y1="-20.32" x2="73.66" y2="-20.32" width="0.1524" layer="91"/>
 <wire x1="73.66" y1="-20.32" x2="73.66" y2="-12.7" width="0.1524" layer="91"/>
@@
 </segment>
 <segment>
-<pinref part="JP1" gate="A" pin="2"/>
+<pinref part="SENSOR.JP" gate="A" pin="2"/>
 <pinref part="P+4" gate="1" pin="+12V"/>
 <wire x1="93.98" y1="-5.08" x2="106.68" y2="-5.08" width="0.1524" layer="91"/>
 <wire x1="106.68" y1="-5.08" x2="106.68" y2="2.54" width="0.1524" layer="91"/>
-<pinref part="JP1" gate="A" pin="8"/>
+<pinref part="SENSOR.JP" gate="A" pin="8"/>
 <wire x1="93.98" y1="-12.7" x2="106.68" y2="-12.7" width="0.1524" layer="91"/>
 <wire x1="106.68" y1="-12.7" x2="106.68" y2="-5.08" width="0.1524" layer="91"/>
-<pinref part="JP1" gate="A" pin="14"/>
+<pinref part="SENSOR.JP" gate="A" pin="14"/>
 <wire x1="93.98" y1="-20.32" x2="106.68" y2="-20.32" width="0.1524" layer="91"/>
 <wire x1="106.68" y1="-20.32" x2="106.68" y2="-12.7" width="0.1524" layer="91"/>
@@
 <net name="SENSOR.LIMIT.X.2" class="0">
 <segment>
-<pinref part="JP1" gate="A" pin="4"/>
+<pinref part="SENSOR.JP" gate="A" pin="4"/>
 <wire x1="93.98" y1="-7.62" x2="114.3" y2="-7.62" width="0.1524" layer="91"/>
 <label x="114.3" y="-7.62" size="0.8128" layer="95" xref="yes"/>
@@
 <net name="SENSOR.LIMIT.Y.2" class="0">
 <segment>
-<pinref part="JP1" gate="A" pin="10"/>
+<pinref part="SENSOR.JP" gate="A" pin="10"/>
 <wire x1="93.98" y1="-15.24" x2="114.3" y2="-15.24" width="0.1524" layer="91"/>
 <label x="114.3" y="-15.24" size="0.8128" layer="95" xref="yes"/>
@@
 <net name="SENSOR.LIMIT.Z.2" class="0">
 <segment>
-<pinref part="JP1" gate="A" pin="16"/>
+<pinref part="SENSOR.JP" gate="A" pin="16"/>
 <wire x1="93.98" y1="-22.86" x2="114.3" y2="-22.86" width="0.1524" layer="91"/>
 <label x="114.3" y="-22.86" size="0.8128" layer="95" xref="yes"/>
@@
 <net name="SENSOR.LIMIT.X.1" class="0">
 <segment>
-<pinref part="JP1" gate="A" pin="3"/>
+<pinref part="SENSOR.JP" gate="A" pin="3"/>
 <wire x1="86.36" y1="-7.62" x2="66.04" y2="-7.62" width="0.1524" layer="91"/>
 <label x="66.04" y="-7.62" size="0.8128" layer="95" rot="R180" xref="yes"/>
@@
 <net name="SENSOR.LIMIT.Y.1" class="0">
 <segment>
-<pinref part="JP1" gate="A" pin="9"/>
+<pinref part="SENSOR.JP" gate="A" pin="9"/>
 <wire x1="86.36" y1="-15.24" x2="66.04" y2="-15.24" width="0.1524" layer="91"/>
 <label x="66.04" y="-15.24" size="0.8128" layer="95" rot="R180" xref="yes"/>
@@
 <net name="SENSOR.LIMIT.Z.1" class="0">
 <segment>
-<pinref part="JP1" gate="A" pin="15"/>
+<pinref part="SENSOR.JP" gate="A" pin="15"/>
 <wire x1="86.36" y1="-22.86" x2="66.04" y2="-22.86" width="0.1524" layer="91"/>
 <label x="66.04" y="-22.86" size="0.8128" layer="95" rot="R180" xref="yes"/>
@@
 </segment>
 </net>
-<net name="+12V" class="0">
+<net name="MEGA2560.VIN.12V" class="0">
 <segment>
 <pinref part="P+2" gate="1" pin="+12V"/>
@@
 </segment>
 </net>
-<net name="GND" class="0">
+<net name="MEGA2560.GND" class="0">
 <segment>
 <pinref part="EXT.JP" gate="A" pin="6"/>
@@
 </busses>
 <nets>
-<net name="GND" class="0">
+<net name="MEGA2560.GND" class="0">
 <segment>
 <pinref part="U$1" gate="G$1" pin="C"/>
@@
 </segment>
 </net>
-<net name="GND" class="0">
+<net name="MEGA2560.GND" class="0">
 <segment>
 <pinref part="U$5" gate="G$1" pin="C"/>
@@
 </segment>
 </net>
-<net name="GND" class="0">
+<net name="MEGA2560.GND" class="0">
 <segment>
 <pinref part="X2" gate="G$1" pin="4"/>
@@
 </segment>
 </net>
+</nets>
+</sheet>
+<sheet>
+<description>Power</description>
+<plain>
+</plain>
+<instances>
+<instance part="GND22" gate="1" x="15.24" y="66.04"/>
+<instance part="P+9" gate="1" x="15.24" y="93.98"/>
+</instances>
+<busses>
+</busses>
+<nets>
+<net name="MEGA2560.VIN.12V" class="0">
+<segment>
+<pinref part="P+9" gate="1" pin="+12V"/>
+<wire x1="15.24" y1="91.44" x2="15.24" y2="83.82" width="0.1524" layer="91"/>
+<wire x1="15.24" y1="83.82" x2="43.18" y2="83.82" width="0.1524" layer="91"/>
+<label x="43.18" y="83.82" size="0.8128" layer="95" xref="yes"/>
+</segment>
+</net>
+<net name="MEGA2560.GND" class="0">
+<segment>
+<pinref part="GND22" gate="1" pin="GND"/>
+<wire x1="15.24" y1="68.58" x2="15.24" y2="76.2" width="0.1524" layer="91"/>
+<wire x1="15.24" y1="76.2" x2="43.18" y2="76.2" width="0.1524" layer="91"/>
+<label x="43.18" y="76.2" size="0.8128" layer="95" xref="yes"/>
+</segment>
+</net>

Commit message: 20180511
Parts:
- removed X1: (no value), con-molex-micro-fit-3_0:HEADER_POS8_43045-0800
- added JP1: (no value), pinhead:PINHD-2X4
- EXT.JP: device pinhead:PINHD-2X11/90 -> pinhead:PINHD-2X11
- SENSOR.JP: device pinhead:PINHD-2X9/90 -> pinhead:PINHD-2X9
- renumbered U$1 to ABORT, U$2 to HOLD, U$3 to START, U$4 to SAFETY.DOOR, U$5 to FLOOD, U$6 to MIST
Connections:
- net +5V: now also JP1.2, JP1.4, JP1.6, JP1.8; no longer X1.1, X1.2, X1.3, X1.4
- net MEGA2560.D8.COOLANT.FLOOD: now also R1.1; no longer LED5.A
- net MEGA2560.D9.COOLANT.MIST: now also R6.1; no longer LED6.A
- net N$19: now also ABORT.A, LED2.C; no longer LED2.A, X1.8
- net N$2: now also LED5.A; no longer FLOOD.A
- net N$20: now also JP1.3, R5.1; no longer LED1.A, X1.7
- net N$21: now also JP1.5, R3.1; no longer LED3.A, X1.6
- net N$22: now also HOLD.A, LED1.C; no longer LED2.C, R4.1
- net N$23: now also LED1.A, R5.2; no longer ABORT.A, R4.2
- net N$24: now also LED2.A, R4.2; no longer HOLD.A, R5.2
- net N$30: now also JP1.1, R4.1; no longer LED1.C, R5.1
- net N$31: now also JP1.7, R2.1; no longer LED4.A, X1.5
- net N$32: now also LED3.A, R3.2; no longer LED3.C, R3.1
- net N$33: now also LED3.C, START.A; no longer LED4.C, R2.1
- net N$34: now also LED4.C; no longer R2.2
- net N$35: now also LED4.A, R2.2; no longer R3.2, START.A
- net N$36: now also LED6.A, R6.2; no longer LED6.C, R6.1
- net N$37: now also LED6.C; no longer MIST.A, R6.2
- net N$4: now also FLOOD.A; no longer R1.1
Other:
- moved on the sheet: LED1, LED2, LED3, LED4, LED5, LED6, R1, R2, R3, R4, R5, R6

Commit message: 20180511
Connections:
- net N$37: now also MIST.A
Changed lines of the file:
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@@
 <segment>
 <pinref part="LED6" gate="G$1" pin="C"/>
-<wire x1="58.42" y1="45.72" x2="71.12" y2="45.72" width="0.1524" layer="91"/>
+<pinref part="MIST" gate="G$1" pin="A"/>
+<wire x1="58.42" y1="45.72" x2="68.58" y2="45.72" width="0.1524" layer="91"/>
 </segment>
 </net>
