File: EAGLE/!PRJ/Control.Board/Control.Board.sch (EAGLE design)
At the start: 55 parts, among them J1 AVR_SPI_PROG_3X2PTH, U1.X LTV817LTV817S, U1.Y LTV817LTV817S, U1.Z LTV817LTV817S, U2.X LTV817LTV817S, U2.Y LTV817LTV817S, U2.Z LTV817LTV817S

Commit message: 20180511
Connections:
- net N$13: now also COOLANT.JP.2; no longer COOLANT.JP.1
- net N$15: now also COOLANT.JP.4; no longer COOLANT.JP.3
- net N$6: now also COOLANT.JP.1; no longer COOLANT.JP.2
- net N$9: now also COOLANT.JP.3; no longer COOLANT.JP.4
Changed lines of the file:
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@@
 <pinref part="FLOOD" gate="G$1" pin="EMIT"/>
 <wire x1="86.36" y1="68.58" x2="91.44" y2="68.58" width="0.1524" layer="91"/>
-<wire x1="91.44" y1="68.58" x2="91.44" y2="71.12" width="0.1524" layer="91"/>
-<pinref part="COOLANT.JP" gate="A" pin="2"/>
-<wire x1="91.44" y1="71.12" x2="109.22" y2="71.12" width="0.1524" layer="91"/>
+<pinref part="COOLANT.JP" gate="A" pin="1"/>
+<wire x1="91.44" y1="68.58" x2="91.44" y2="73.66" width="0.1524" layer="91"/>
+<wire x1="91.44" y1="73.66" x2="109.22" y2="73.66" width="0.1524" layer="91"/>
 </segment>
 </net>
@@
 <pinref part="MIST" gate="G$1" pin="EMIT"/>
 <wire x1="86.36" y1="40.64" x2="96.52" y2="40.64" width="0.1524" layer="91"/>
-<wire x1="96.52" y1="40.64" x2="96.52" y2="66.04" width="0.1524" layer="91"/>
-<pinref part="COOLANT.JP" gate="A" pin="4"/>
-<wire x1="96.52" y1="66.04" x2="109.22" y2="66.04" width="0.1524" layer="91"/>
+<pinref part="COOLANT.JP" gate="A" pin="3"/>
+<wire x1="96.52" y1="40.64" x2="96.52" y2="68.58" width="0.1524" layer="91"/>
+<wire x1="96.52" y1="68.58" x2="109.22" y2="68.58" width="0.1524" layer="91"/>
 </segment>
 </net>
@@
 </segment>
 </net>
-<net name="N$13" class="0">
-<segment>
-<pinref part="FLOOD" gate="G$1" pin="COL"/>
-<pinref part="COOLANT.JP" gate="A" pin="1"/>
-<wire x1="86.36" y1="73.66" x2="109.22" y2="73.66" width="0.1524" layer="91"/>
-</segment>
-</net>
 <net name="N$15" class="0">
 <segment>
-<pinref part="COOLANT.JP" gate="A" pin="3"/>
-<wire x1="109.22" y1="68.58" x2="93.98" y2="68.58" width="0.1524" layer="91"/>
-<wire x1="93.98" y1="68.58" x2="93.98" y2="45.72" width="0.1524" layer="91"/>
 <pinref part="MIST" gate="G$1" pin="COL"/>
 <wire x1="93.98" y1="45.72" x2="86.36" y2="45.72" width="0.1524" layer="91"/>
+<pinref part="COOLANT.JP" gate="A" pin="4"/>
+<wire x1="93.98" y1="45.72" x2="93.98" y2="66.04" width="0.1524" layer="91"/>
+<wire x1="93.98" y1="66.04" x2="109.22" y2="66.04" width="0.1524" layer="91"/>
 </segment>
 </net>
@@
 </segment>
 </net>
+<net name="N$13" class="0">
+<segment>
+<pinref part="FLOOD" gate="G$1" pin="COL"/>
+<pinref part="COOLANT.JP" gate="A" pin="2"/>
+<wire x1="86.36" y1="73.66" x2="86.36" y2="71.12" width="0.1524" layer="91"/>
+<wire x1="86.36" y1="71.12" x2="109.22" y2="71.12" width="0.1524" layer="91"/>
+</segment>
+</net>

Commit message: 20180513
Parts:
- PROBE: device pinhead:PINHD-1X2/90 -> pinhead:PINHD-1X2
Connections:
- new net GND: ABORT.C, HOLD.C, PROBE.1, SAFETY.DOOR.C, START.C
- new net MEGA2560.GND.INT.1: JP.MEGA2560.PWM.HIGH.4
- net MEGA2560.A15.PROBE: now also PROBE.2; no longer PROBE.1
- net MEGA2560.GND: no longer ABORT.C, HOLD.C, JP.MEGA2560.PWM.HIGH.4, PROBE.2, SAFETY.DOOR.C, START.C
Other:
- moved on the sheet: PROBE

Commit message: Auto stash before merge of "master" and "origin/master"
Parts:
- removed J1: AVR_SPI_PROG_3X2PTH, SparkFun-Connectors:AVR_SPI_PROG_3X2PTH
Changed lines of the file:
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@@
 <part name="JP.MEGA2560.COMMUNICATION" library="pinhead" deviceset="PINHD-1X8" device=""/>
 <part name="JP.MEGA2560.PWM.LOW" library="pinhead" deviceset="PINHD-1X8" device=""/>
-<part name="J1" library="SparkFun-Connectors" deviceset="AVR_SPI_PROG_3X2" device="PTH"/>
 <part name="U1.X" library="net173" deviceset="LTV817" device="LTV817S"/>
 <part name="U2.X" library="net173" deviceset="LTV817" device="LTV817S"/>
@@
 <instance part="JP.MEGA2560.COMMUNICATION" gate="A" x="66.04" y="27.94" rot="MR0"/>
 <instance part="JP.MEGA2560.PWM.LOW" gate="A" x="66.04" y="55.88" rot="MR0"/>
-<instance part="J1" gate="G$1" x="132.08" y="50.8"/>
 </instances>
 <busses>
